Commit message: First sim champ implementation

File: src/go2_sim/urdf/go2_sim.urdf.xacro (robot description, xacro)
@@ -2,263 +2,247 @@
 <!--
   go2_sim.urdf.xacro
-  Unitree Go2 - Gazebo Classic (Gazebo 11) simulation model.
-  This model keeps the detailed Go2 visuals while preserving the planar-move
-  physics contract that the old working simulation relied on:
-    - Visual-only legs and sensor pods for appearance
-    - A simplified torso collision plus a flat contact proxy for stable planar motion
-    - Unchanged Nav2-facing topics and frames
+  Unitree Go2 — Gazebo Fortress (Ignition Gazebo 6) + CHAMP simulation model.
+  Port contract:
+    - Source:  khaledgabr77/unitree_go2_ros2 (Gazebo Harmonic, ROS 2 Jazzy)
+    - Target:  go2_sim (Gazebo Fortress / Ignition Gazebo 6, ROS 2 Humble)
+  Frame tree:
+    base_link (robot body — matches go2_description and go2_bringup convention)
+      ├── trunk                  (body visual/collision/inertia; floating_base joint)
+      ├── imu_link               (IMU sensor frame)
+      ├── {lf,rf,lh,rh}_hip_link → {lf,rf,lh,rh}_upper_leg_link
+      │                         → {lf,rf,lh,rh}_lower_leg_link
+      │                         → LF_FOOT / RF_FOOT / LH_FOOT / RH_FOOT (CHAMP)
+      └── lidar_l1_link          (Unitree L1 LiDAR; provided by sensor_models macro)
+  CHAMP requires four foot links named exactly: LF_FOOT RF_FOOT LH_FOOT RH_FOOT
+  These are generated by the leg macro in leg.xacro.
+  Fortress plugins used (all Classic libgazebo_ros_* plugins removed):
+    - ign_ros2_control-system          (joint trajectory effort control)
+    - ignition-gazebo-imu-system       (IMU sensor)
+    - ignition-gazebo-contact-system   (foot contact sensors)
+    - ignition-gazebo-joint-state-publisher-system  (/joint_states)
+    - ignition-gazebo-sensors-system   (gpu_lidar — in world SDF, handles L1)
+  Topics published (bridged to ROS via ros_ign_bridge in launch file):
+    /joint_states       — sensor_msgs/JointState
+    /imu/data           — sensor_msgs/Imu
+    /lidar/points     — sensor_msgs/PointCloud2   (from L1 lidar_l1 sensor)
+    /cmd_vel            — geometry_msgs/Twist        (ROS → Gazebo)
+  DO NOT USE libgazebo_ros_* plugins here — they are Gazebo Classic only.
+  DO NOT USE gz:: namespaces — Fortress uses ignition:: exclusively.
 -->
-<robot name="go2_sim" xmlns:xacro="http://www.ros.org/wiki/xacro">
+<robot name="go2"
+       xmlns:xacro="http://www.ros.org/wiki/xacro">
+  <!-- ── xacro arguments ── -->
+  <xacro:arg name="DEBUG"            default="false"/>
+  <xacro:arg name="robot_controllers"
+             default="$(find go2_sim)/config/ros_control.yaml"/>
+  <!-- ── Include sub-files ── -->
+  <xacro:include filename="$(find go2_sim)/urdf/const.xacro"/>
+  <xacro:include filename="$(find go2_sim)/urdf/materials.xacro"/>
+  <xacro:include filename="$(find go2_sim)/urdf/leg.xacro"/>
   <xacro:include filename="$(find sensor_models)/urdf/l1_lidar.urdf.xacro"/>
-  <xacro:property name="mesh_pkg" value="go2_sim"/>
-  <xacro:property name="trunk_length" value="0.3762"/>
-  <xacro:property name="trunk_width" value="0.0935"/>
-  <xacro:property name="trunk_height" value="0.114"/>
-  <xacro:property name="trunk_mass" value="6.921"/>
-  <!-- Keep the planar-move physics frame at the old stable height.
-       Detailed visuals are offset separately so the rendered model still
-       matches the newer Go2 appearance without raising the COM. -->
-  <xacro:property name="base_z" value="0.335"/>
-  <xacro:property name="visual_z_offset" value="0.045"/>
-  <xacro:property name="contact_proxy_length" value="0.5794"/>
-  <xacro:property name="contact_proxy_width" value="0.328"/>
-  <xacro:property name="contact_proxy_height" value="0.020"/>
-  <xacro:property name="contact_proxy_z" value="${-(base_z - (contact_proxy_height * 0.5))}"/>
-  <xacro:property name="q_hip" value="0.0"/>
-  <xacro:property name="q_thigh" value="0.67"/>
-  <xacro:property name="q_calf" value="-1.30"/>
-  <!-- Lidar mount point (from khaledgabr77/unitree_go2_ros2 reference).
-       The joint uses ${lidar_z + visual_z_offset}, so lidar_z = -0.03 - 0.045 = -0.075
-       to place the sensor at z=-0.03 relative to base_link (same as reference). -->
-  <xacro:property name="lidar_x" value="0.25"/>
-  <xacro:property name="lidar_y" value="-0.038"/>
-  <xacro:property name="lidar_z" value="-0.075"/>
-  <xacro:property name="lidar_r" value="0.0"/>
-  <xacro:property name="lidar_p" value="0.0"/>
-  <xacro:property name="lidar_yaw" value="0.0"/>
-  <xacro:macro name="go2_leg_visual" params="
-      prefix
-      hip_x
-      hip_y
-      thigh_y
-      hip_visual_rpy
-      thigh_mesh
-      calf_mesh">
-    <link name="${prefix}_hip">
-      <visual>
-        <origin xyz="0 0 0" rpy="${hip_visual_rpy}"/>
-        <geometry>
-          <mesh filename="package://${mesh_pkg}/meshes/dae/hip.dae"/>
-        </geometry>
-      </visual>
-    </link>
-    <joint name="${prefix}_hip_joint" type="fixed">
-      <origin xyz="${hip_x} ${hip_y} ${visual_z_offset}" rpy="${q_hip} 0 0"/>
-      <parent link="base_link"/>
-      <child link="${prefix}_hip"/>
+  <!-- ════════════════════════════════════════════════════════════════════
+       GAZEBO PLUGINS  (Fortress / ignition:: namespace)
+       ════════════════════════════════════════════════════════════════════ -->
+  <!-- ign_ros2_control: loads controller_manager, reads ros_control.yaml -->
+  <gazebo>
+    <plugin filename="ign_ros2_control-system"
+            name="ign_ros2_control::IgnitionROS2ControlPlugin">
+      <parameters>$(arg robot_controllers)</parameters>
+      <robot_param_node>robot_state_publisher</robot_param_node>
+    </plugin>
+  </gazebo>
+  <!-- Joint state publisher: publishes /joint_states from sim -->
+  <gazebo>
+    <plugin filename="ignition-gazebo-joint-state-publisher-system"
+            name="ignition::gazebo::systems::JointStatePublisher">
+    </plugin>
+  </gazebo>
+  <!-- ════════════════════════════════════════════════════════════════════
+       OPTIONAL DEBUG MODE: pin robot to world for tuning
+       ════════════════════════════════════════════════════════════════════ -->
+  <xacro:if value="$(arg DEBUG)">
+    <link name="world"/>
+    <joint name="base_static_joint" type="fixed">
+      <origin rpy="0 0 0" xyz="0 0 0"/>
+      <parent link="world"/>
+      <child link="base_link"/>
     </joint>
-    <link name="${prefix}_thigh">
-      <visual>
-        <origin xyz="0 0 0" rpy="0 0 0"/>
-        <geometry>
-          <mesh filename="package://${mesh_pkg}/meshes/dae/${thigh_mesh}"/>
-        </geometry>
-      </visual>
-    </link>
-    <joint name="${prefix}_thigh_joint" type="fixed">
-      <origin xyz="0 ${thigh_y} 0" rpy="0 ${q_thigh} 0"/>
-      <parent link="${prefix}_hip"/>
-      <child link="${prefix}_thigh"/>
-    </joint>
-    <link name="${prefix}_calf">
-      <visual>
-        <origin xyz="0 0 0" rpy="0 0 0"/>
-        <geometry>
-          <mesh filename="package://${mesh_pkg}/meshes/dae/${calf_mesh}"/>
-        </geometry>
-      </visual>
-    </link>
-    <joint name="${prefix}_calf_joint" type="fixed">
-      <origin xyz="0 0 -0.213" rpy="0 ${q_calf} 0"/>
-      <parent link="${prefix}_thigh"/>
-      <child link="${prefix}_calf"/>
-    </joint>
-    <link name="${prefix}_foot">
-      <visual>
-        <origin xyz="0 0 0" rpy="0 0 0"/>
-        <geometry>
-          <mesh filename="package://${mesh_pkg}/meshes/dae/foot.dae"/>
-        </geometry>
-      </visual>
-    </link>
-    <joint name="${prefix}_foot_joint" type="fixed">
-      <origin xyz="0 0 -0.213" rpy="0 0 0"/>
-      <parent link="${prefix}_calf"/>
-      <child link="${prefix}_foot"/>
-    </joint>
-  </xacro:macro>
-  <link name="base_footprint">
+  </xacro:if>
+  <!-- ════════════════════════════════════════════════════════════════════
+       BASE LINK  (virtual root — matches CHAMP expectation)
+       ════════════════════════════════════════════════════════════════════ -->
+  <link name="base_link">
     <visual>
+      <origin rpy="0 0 0" xyz="0 0 0"/>
       <geometry><box size="0.001 0.001 0.001"/></geometry>
     </visual>
   </link>
-  <joint name="base_footprint_to_base_link" type="fixed">
-    <parent link="base_footprint"/>
-    <child link="base_link"/>
-    <origin xyz="0 0 ${base_z}" rpy="0 0 0"/>
+  <!-- ════════════════════════════════════════════════════════════════════
+       TRUNK  (main body visual / collision / inertia)
+       Mesh: base.dae  (byte-identical to source trunk.dae; same 10727399 B)
+       ════════════════════════════════════════════════════════════════════ -->
+  <joint name="floating_base" type="fixed">
+    <origin rpy="0 0 0" xyz="0 0 0"/>
+    <parent link="base_link"/>
+    <child link="trunk"/>
   </joint>
-  <link name="base_link">
-    <inertial>
-      <origin xyz="0.021112 0 -0.005366" rpy="0 0 0"/>
-      <mass value="${trunk_mass}"/>
-      <inertia ixx="0.02448" ixy="0.00012166" ixz="0.0014849" iyy="0.098077" iyz="-3.12E-05" izz="0.107"/>
-    </inertial>
+  <link name="trunk">
     <visual>
-      <origin xyz="0 0 ${visual_z_offset}" rpy="0 0 0"/>
+      <origin rpy="0 0 0" xyz="0 0 0"/>
       <geometry>
-        <mesh filename="package://${mesh_pkg}/meshes/dae/base.dae"/>
+        <mesh filename="package://go2_sim/meshes/dae/base.dae" scale="1 1 1"/>
       </geometry>
     </visual>
     <collision>
-      <origin xyz="0 0 0" rpy="0 0 0"/>
+      <origin rpy="0 0 0" xyz="0 0 0"/>
       <geometry>
         <box size="${trunk_length} ${trunk_width} ${trunk_height}"/>
       </geometry>
     </collision>
-    <collision>
-      <origin xyz="0 0 ${contact_proxy_z}" rpy="0 0 0"/>
-      <geometry>
-        <box size="${contact_proxy_length} ${contact_proxy_width} ${contact_proxy_height}"/>
-      </geometry>
-    </collision>
+    <inertial>
+      <origin rpy="0 0 0" xyz="${trunk_com_x} ${trunk_com_y} ${trunk_com_z}"/>
+      <mass value="${trunk_mass}"/>
+      <inertia ixx="${trunk_ixx}" ixy="${trunk_ixy}" ixz="${trunk_ixz}"
+               iyy="${trunk_iyy}" iyz="${trunk_iyz}" izz="${trunk_izz}"/>
+    </inertial>
   </link>
-  <xacro:go2_leg_visual
-      prefix="FL"
-      hip_x="0.1934"
-      hip_y="0.0465"
-      thigh_y="0.0955"
-      hip_visual_rpy="0 0 0"
-      thigh_mesh="thigh.dae"
-      calf_mesh="calf.dae"/>
-  <xacro:go2_leg_visual
-      prefix="FR"
-      hip_x="0.1934"
-      hip_y="-0.0465"
-      thigh_y="-0.0955"
-      hip_visual_rpy="3.141592653589793 0 0"
-      thigh_mesh="thigh_mirror.dae"
-      calf_mesh="calf_mirror.dae"/>
-  <xacro:go2_leg_visual
-      prefix="RL"
-      hip_x="-0.1934"
-      hip_y="0.0465"
-      thigh_y="0.0955"
-      hip_visual_rpy="0 3.141592653589793 0"
-      thigh_mesh="thigh.dae"
-      calf_mesh="calf.dae"/>
-  <xacro:go2_leg_visual
-      prefix="RR"
-      hip_x="-0.1934"
-      hip_y="-0.0465"
-      thigh_y="-0.0955"
-      hip_visual_rpy="3.141592653589793 3.141592653589793 0"
-      thigh_mesh="thigh_mirror.dae"
-      calf_mesh="calf_mirror.dae"/>
+  <gazebo reference="trunk">
+    <mu1>0.2</mu1>
+    <mu2>0.2</mu2>
+    <kp>10000.0</kp>
+    <kd>1.0</kd>
+  </gazebo>
+  <!-- ════════════════════════════════════════════════════════════════════
+       IMU LINK
+       ════════════════════════════════════════════════════════════════════ -->
   <joint name="imu_joint" type="fixed">
-    <origin xyz="-0.02557 0 ${0.04232 + visual_z_offset}" rpy="0 0 0"/>
-    <parent link="base_link"/>
+    <parent link="trunk"/>
     <child link="imu_link"/>
+    <origin rpy="0 0 0" xyz="0 0 0"/>
   </joint>
   <link name="imu_link">
     <inertial>
       <mass value="0.001"/>
-      <origin xyz="0 0 0" rpy="0 0 0"/>
-      <inertia ixx="1e-7" ixy="0" ixz="0" iyy="1e-7" iyz="0" izz="1e-7"/>
+      <origin rpy="0 0 0" xyz="0 0 0"/>
+      <inertia ixx="0.0001" ixy="0" ixz="0" iyy="0.0001" iyz="0" izz="0.0001"/>
     </inertial>
+    <visual>
+      <origin rpy="0 0 0" xyz="0 0 0"/>
+      <geometry><box size="0.001 0.001 0.001"/></geometry>
+    </visual>
+    <collision>
+      <origin rpy="0 0 0" xyz="0 0 0"/>
+      <geometry><box size="0.001 0.001 0.001"/></geometry>
+    </collision>
   </link>
-  <joint name="radar_joint" type="fixed">
-    <origin xyz="0.28945 0 ${-0.046825 + visual_z_offset}" rpy="0 2.8782 0"/>
-    <parent link="base_link"/>
-    <child link="radar"/>
-  </joint>
-  <link name="radar"/>
-  <joint name="front_camera_joint" type="fixed">
-    <origin xyz="0.32715 -0.00003 ${0.04297 + visual_z_offset}" rpy="0 0 0"/>
-    <parent link="base_link"/>
-    <child link="front_camera_link"/>
-  </joint>
-  <link name="front_camera_link"/>
-  <joint name="base_link_to_lidar" type="fixed">
-    <parent link="base_link"/>
-    <child link="lidar_link"/>
-    <origin xyz="${lidar_x} ${lidar_y} ${lidar_z + visual_z_offset}" rpy="${lidar_r} ${lidar_p} ${lidar_yaw}"/>
-  </joint>
-  <link name="lidar_link">
-    <visual>
-      <origin xyz="0 0 0" rpy="0 0 0"/>
-      <geometry>
-        <cylinder radius="0.04" length="0.06"/>
-      </geometry>
-      <material name="lidar_black">
-        <color rgba="0.05 0.05 0.05 1.0"/>
-      </material>
-    </visual>
-    <inertial>
-      <mass value="0.001"/>
-      <origin xyz="0 0 0" rpy="0 0 0"/>
-      <inertia ixx="1e-7" ixy="0" ixz="0" iyy="1e-7" iyz="0" izz="1e-7"/>
-    </inertial>
-  </link>
-  <gazebo reference="base_link">
-    <material>Gazebo/DarkGrey</material>
-    <self_collide>false</self_collide>
-    <mu1>0.8</mu1>
-    <mu2>0.8</mu2>
-  </gazebo>
-  <gazebo reference="lidar_link">
-    <material>Gazebo/Black</material>
-  </gazebo>
-  <gazebo>
-    <plugin name="gazebo_ros_planar_move" filename="libgazebo_ros_planar_move.so">
-      <ros>
-        <remapping>cmd_vel:=/cmd_vel</remapping>
-        <remapping>odom:=/odom</remapping>
-      </ros>
-      <update_rate>50</update_rate>
-      <publish_odom>true</publish_odom>
-      <publish_odom_tf>true</publish_odom_tf>
-      <odometry_frame>odom</odometry_frame>
-      <robot_base_frame>base_footprint</robot_base_frame>
-      <covariance_x>0.0001</covariance_x>
-      <covariance_y>0.0001</covariance_y>
-      <covariance_yaw>0.01</covariance_yaw>
-    </plugin>
-  </gazebo>
-  <!-- L1 sensor parameters from khaledgabr77/unitree_go2_ros2 reference:
-       600 h-samples, 30 v-channels, range 0.8–30 m, noise σ=0.008 m. -->
-  <xacro:l1_lidar_gazebo
-      parent_link="lidar_link"
-      topic="/unilidar/cloud"
-      update_rate="10"
-      h_samples="600"
-      v_samples="30"
-      v_min_angle_deg="-45.0"
-      v_max_angle_deg="45.0"
-      range_min="0.8"
-      range_max="30.0"
-      noise_stddev="0.008"
-      visualize="false"
-  />
+  <!--
+    IMU sensor (Fortress syntax).
+    Published on topic: /imu/data
+    Bridged to ROS via ros_ign_bridge in sim_champ.launch.py.
+    System plugin ignition-gazebo-imu-system is loaded in the world SDF.
+  -->
   <gazebo reference="imu_link">
-    <sensor type="imu" name="go2_imu">
-      <always_on>true</always_on>
-      <update_rate>250</update_rate>
-      <plugin name="gazebo_ros_imu" filename="libgazebo_ros_imu_sensor.so">
-        <ros>
-          <remapping>~/out:=/unilidar/imu</remapping>
-        </ros>
-        <initial_orientation_as_reference>false</initial_orientation_as_reference>
-      </plugin>
-    </sensor>
-  </gazebo>
+    <sensor name="imu_sensor" type="imu">
+      <always_on>1</always_on>
+      <update_rate>200</update_rate>
+      <topic>/imu/data</topic>
+      <ignition_frame_id>imu_link</ignition_frame_id>
+      <imu>
+        <angular_velocity>
+          <x><noise type="gaussian"><mean>0</mean><stddev>0.009</stddev></noise></x>
+          <y><noise type="gaussian"><mean>0</mean><stddev>0.009</stddev></noise></y>
+          <z><noise type="gaussian"><mean>0</mean><stddev>0.009</stddev></noise></z>
+        </angular_velocity>
+        <linear_acceleration>
+          <x><noise type="gaussian"><mean>0</mean><stddev>0.021</stddev></noise></x>
+          <y><noise type="gaussian"><mean>0</mean><stddev>0.021</stddev></noise></y>
+          <z><noise type="gaussian"><mean>0</mean><stddev>0.021</stddev></noise></z>
+        </linear_acceleration>
+      </imu>
+    </sensor>
+  </gazebo>
+  <!-- ════════════════════════════════════════════════════════════════════
+       LEGS  (4× instantiation via leg macro — defines foot links LF/RF/LH/RH_FOOT)
+       ════════════════════════════════════════════════════════════════════ -->
+  <!--  RF: mirror=-1 (right), mirror_dae=False (right mesh), front_hind=1, front_hind_dae=True  -->
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