Commit message: First sim champ implementation

File: src/sensor_models/urdf/l1_lidar.urdf.xacro (robot description, xacro)
@@ -2,34 +2,129 @@
 <!--
   l1_lidar.urdf.xacro
-  Reusable Gazebo Classic (Gazebo 11) macro for the Unitree L1 LiDAR sensor.
+  Reusable sensor macros for the Unitree L1 LiDAR sensor.
+  Two macros are provided:
+    1. l1_lidar          — Gazebo Fortress (Ignition Gazebo 6, ROS 2 Humble) — USE THIS
+    2. l1_lidar_gazebo   — Gazebo Classic (Gazebo 11) — kept for robot_sim Classic pipeline
+  ─────────────────────────────────────────────────────────────────────────────
+  MACRO: l1_lidar  (Fortress / Ignition Gazebo 6)
+  ─────────────────────────────────────────────────────────────────────────────
   Unitree L1 device specifications (from Unitree datasheet):
-    - Scan lines (vertical channels): 18
+    - Scan lines (vertical channels): 18 (simulation uses 30 for fidelity)
     - Vertical FOV: ±45° (−45° to +45°)
     - Horizontal FOV: 360°
     - Rotation frequency (typical): 10 Hz
-    - Range: 0.05 m – 30 m
-    - Simulation default horizontal samples: 360 (1 sample per degree)
+    - Range: 0.8 m – 30 m
+    - Simulation noise σ: 0.008 m
   Usage:
     <xacro:include filename="$(find sensor_models)/urdf/l1_lidar.urdf.xacro"/>
+    <xacro:l1_lidar parent="base_link" prefix="">
+      <origin xyz="0.25 -0.038 -0.03" rpy="0 0 0"/>
+    </xacro:l1_lidar>
+  Parameters:
+    parent  — URDF link to attach the lidar link to (required)
+    prefix  — string prepended to all generated link/joint/sensor names (may be "")
+  Block parameter:
+    *origin — <origin xyz="..." rpy="..."/> child element (required)
+  The macro creates:
+    - Link:  ${prefix}lidar_link  (named for nav stack compatibility: scan_from_cloud.yaml
+             expects target_frame: lidar_link; with prefix="" this yields "lidar_link")
+    - Joint: ${prefix}lidar_l1_joint  (fixed, parent→child, origin from block)
+    - Gazebo gpu_lidar sensor on ${prefix}lidar_link
+      Gazebo topics:
+        /unilidar/cloud         (LaserScan)
+        /unilidar/cloud/points  (PointCloudPacked, bridged to ROS /lidar/points)
+  ─────────────────────────────────────────────────────────────────────────────
+  MACRO: l1_lidar_gazebo  (Classic / Gazebo 11) — legacy, do not use for Fortress
+  ─────────────────────────────────────────────────────────────────────────────
+  Usage:
     <xacro:l1_lidar_gazebo parent_link="lidar_link"/>
-  Optional overrides (all have defaults matching L1 specs):
-    topic           — PointCloud2 output topic (default: /unilidar/cloud)
-    update_rate     — scan frequency in Hz          (default: 10)
-    h_samples       — horizontal rays per line       (default: 360)
-    v_samples       — vertical channels              (default: 18)
-    v_min_angle_deg — lower vertical angle in deg    (default: -45.0)
-    v_max_angle_deg — upper vertical angle in deg    (default:  45.0)
-    range_min       — minimum valid range in m       (default: 0.05)
-    range_max       — maximum valid range in m       (default: 30.0)
-    noise_stddev    — range noise std deviation in m (default: 0.02)
-    visualize       — show ray visualisation in Rviz (default: false)
-  Porting note (TODO(agibot)):
-    AgiBot D1 Ultra uses a different LiDAR.  Add a separate macro (e.g. d1_lidar_gazebo)
-    or override the parameters to match D1 specs when porting.
 -->
 <robot xmlns:xacro="http://www.ros.org/wiki/xacro">
+  <!-- ═══════════════════════════════════════════════════════════════════════
+       FORTRESS MACRO  (ignition-gazebo-sensors-system handles the sensor)
+       ═══════════════════════════════════════════════════════════════════════ -->
+  <xacro:macro name="l1_lidar" params="
+      parent
+      prefix
+      range_min:=0.8
+      range_max:=30.0
+      *origin">
+    <link name="${prefix}lidar_link">
+      <visual>
+        <origin xyz="0 0 0" rpy="0 0 0"/>
+        <geometry>
+          <cylinder radius="0.04" length="0.05"/>
+        </geometry>
+        <material name="lidar_black">
+          <color rgba="0.05 0.05 0.05 1.0"/>
+        </material>
+      </visual>
+      <inertial>
+        <mass value="0.5"/>
+        <origin xyz="0 0 0" rpy="0 0 0"/>
+        <inertia ixx="0.001" ixy="0" ixz="0" iyy="0.001" iyz="0" izz="0.001"/>
+      </inertial>
+    </link>
+    <joint name="${prefix}lidar_l1_joint" type="fixed">
+      <parent link="${parent}"/>
+      <child link="${prefix}lidar_link"/>
+      <xacro:insert_block name="origin"/>
+    </joint>
+    <!--
+      Fortress gpu_lidar sensor.
+      The sensor system is loaded in the world SDF via:
+        ignition-gazebo-sensors-system  (ignition::gazebo::systems::Sensors)
+      No per-sensor plugin element is required.
+      ignition_frame_id: sets the ROS frame_id in the bridged PointCloud2 message.
+      With prefix="" this yields "lidar_link" which matches scan_from_cloud.yaml
+      (target_frame: lidar_link) and go2_description/go2_bringup conventions.
+      PointCloud topic /unilidar/cloud/points is bridged by ros_ign_bridge
+      in the launch file to ROS topic /lidar/points.
+    -->
+    <gazebo reference="${prefix}lidar_link">
+      <sensor name="${prefix}lidar_l1" type="gpu_lidar">
+        <topic>/unilidar/cloud</topic>
+        <update_rate>10</update_rate>
+        <always_on>1</always_on>
+        <visualize>false</visualize>
+        <ignition_frame_id>${prefix}lidar_link</ignition_frame_id>
+        <ray>
+          <scan>
+            <horizontal>
+              <!-- 360° sweep -->
+              <samples>600</samples>
+              <resolution>1</resolution>
+              <min_angle>-3.14159265358979</min_angle>
+              <max_angle>3.14159265358979</max_angle>
+            </horizontal>
+            <vertical>
+              <!-- ±45° vertical FOV, 30 channels -->
+              <samples>30</samples>
+              <resolution>1</resolution>
+              <min_angle>-0.78539816339745</min_angle>
+              <max_angle>0.78539816339745</max_angle>
+            </vertical>
+          </scan>
+          <range>
+            <min>${range_min}</min>
+            <max>${range_max}</max>
+            <resolution>0.001</resolution>
+          </range>
+          <noise>
+            <type>gaussian</type>
+            <mean>0.0</mean>
+            <stddev>0.008</stddev>
+          </noise>
+        </ray>
+      </sensor>
+    </gazebo>
+  </xacro:macro>
+  <!-- ═══════════════════════════════════════════════════════════════════════
+       CLASSIC MACRO  (Gazebo 11 / libgazebo_ros_ray_sensor)
+       Kept for the robot_sim Gazebo Classic pipeline.  Do NOT use in Fortress.
+       ═══════════════════════════════════════════════════════════════════════ -->
   <xacro:macro name="l1_lidar_gazebo" params="
       parent_link
-      topic:='/unilidar/cloud'
+      topic:='/lidar/points'
       update_rate:=10
       h_samples:=360
@@ -37,19 +132,12 @@
       v_min_angle_deg:=-45.0
       v_max_angle_deg:=45.0
-      range_min:=0.05
+      range_min:=0.15
       range_max:=30.0
       noise_stddev:=0.02
       visualize:=false
   ">
-    <!-- Convert vertical angles from degrees to radians using xacro arithmetic -->
     <xacro:property name="deg_to_rad" value="${pi / 180.0}"/>
     <xacro:property name="v_min_rad"  value="${v_min_angle_deg * deg_to_rad}"/>
     <xacro:property name="v_max_rad"  value="${v_max_angle_deg * deg_to_rad}"/>
-    <!--
-      Use gpu_ray for hardware-accelerated multi-beam LiDAR simulation.
-      Falls back to 'ray' on CPU-only systems — change the sensor type attribute
-      and the plugin filename from libgazebo_ros_ray_sensor.so to the same name
-      (the plugin supports both sensor types).
-    -->
     <gazebo reference="${parent_link}">
       <sensor type="gpu_ray" name="l1_lidar">
@@ -60,5 +148,4 @@
           <scan>
             <horizontal>
-              <!-- 360° sweep. min_angle = -π, max_angle = +π -->
               <samples>${h_samples}</samples>
               <resolution>1</resolution>
@@ -76,5 +163,4 @@
             <min>${range_min}</min>
             <max>${range_max}</max>
-            <!-- sub-cm depth resolution -->
             <resolution>0.001</resolution>
           </range>
@@ -85,9 +171,4 @@
           </noise>
         </ray>
-        <!--
-          gazebo_ros_ray_sensor (gazebo_plugins, Apache-2.0)
-          Publishes sensor_msgs/PointCloud2 on ${topic}.
-          frame_name must match the URDF link referenced by this <gazebo> block.
-        -->
         <plugin name="gazebo_ros_l1_lidar" filename="libgazebo_ros_ray_sensor.so">
           <ros>
