Commit message: Improved Gazebo Go2 Model

File: src/go2_description/urdf/go2.urdf.xacro (robot description, xacro)
@@ -40,8 +40,12 @@
   <!-- Nominal standing torso centre height from ground [m]. -->
   <xacro:property name="standing_height" value="0.28"/>
-  <!-- Front-top sensor mount from root official go2.urdf Head_upper_joint. -->
-  <xacro:property name="lidar_x" value="0.285"/>
+  <!-- Front-top sensor mount matching official Unitree Go2 radar_joint -->
+  <xacro:property name="lidar_x" value="0.28945"/>
   <xacro:property name="lidar_y" value="0.0"/>
-  <xacro:property name="lidar_z" value="0.01"/>
+  <xacro:property name="lidar_z" value="-0.046825"/>
+  <xacro:property name="lidar_r" value="0.0"/>
+  <!-- <xacro:property name="lidar_p" value="2.8782"/> -->
+  <xacro:property name="lidar_p" value="0.0"/>
+  <xacro:property name="lidar_yaw" value="0.0"/>
   <!-- ═══════════════════════════════════════════════════════════════════════
        base_footprint  —  ground contact reference (Nav2 global frame anchor)
@@ -141,5 +145,5 @@
     <parent link="base_link"/>
     <child  link="lidar_link"/>
-    <origin xyz="${lidar_x} ${lidar_y} ${lidar_z}" rpy="0 0 0"/>
+    <origin xyz="${lidar_x} ${lidar_y} ${lidar_z}" rpy="${lidar_r} ${lidar_p} ${lidar_yaw}"/>
   </joint>
   <link name="lidar_link">

File: src/go2_sim/urdf/go2_sim.urdf.xacro (robot description, xacro)
@@ -2,97 +2,715 @@
 <!--
   go2_sim.urdf.xacro
-  Unitree Go2 — Gazebo Classic (Gazebo 11) simulation model.
-  Standalone file: does NOT xacro:include go2_description.  Both can be used side-by-side.
-  Frame tree (identical to go2_description/urdf/go2.urdf.xacro):
-    base_footprint  (ground projection; Nav2 2D footprint frame)
-      └─ base_link        (robot trunk centre, z = 0.335 m above ground)
-           ├─ imu_link     (co-located with trunk; Gazebo IMU sensor)
-           └─ lidar_link   (Unitree L1 LiDAR forward-top mount)
-  Gazebo plugins:
-    libgazebo_ros_planar_move — subscribes /cmd_vel, publishes /odom + TF(odom→base_footprint)
-                                 replaces go2_hw_bridge; Nav2 sees exactly the same interface.
-    L1 LiDAR GPU ray sensor  — publishes /unilidar/cloud (PointCloud2, 10 Hz, 18 lines)
-                                 via sensor_models/l1_lidar_gazebo xacro macro.
-    IMU sensor               — publishes /unilidar/imu (sensor_msgs/Imu, 250 Hz)
-  Physical parameters match go2_description (same trunk dimensions, inertia, sensor positions).
-  TODO(agibot): For AgiBot D1 Ultra, create agibot_d1_sim/urdf/d1_sim.urdf.xacro with:
-    - Same frame names
-    - D1 Ultra chassis dimensions and inertia
-    - Replace L1 LiDAR macro call with D1's sensor macro (add to sensor_models/)
-    - Keep the planar_move plugin block unchanged
+  Unitree Go2 - Gazebo Classic (Gazebo 11) simulation model.
+  Visual model: official Unitree meshes from
+    https://github.com/unitreerobotics/unitree_ros/tree/master/robots/go2_description
+  Leg joints are fixed at the nominal standing pose:
+    hip=0.0 rad, thigh=0.67 rad, calf=-1.30 rad.
+  This keeps the robot visually correct while avoiding joint-control instability.
+  The planar_move plugin still drives locomotion via /cmd_vel as before.
+  Frame tree:
+    base_footprint (ground reference, Nav2 root)
+      -> base_link (maps to upstream link "base")
+         -> FL_hip -> FL_thigh -> FL_calf -> FL_foot
+         -> FR_hip -> FR_thigh -> FR_calf -> FR_foot
+         -> RL_hip -> RL_thigh -> RL_calf -> RL_foot
+         -> RR_hip -> RR_thigh -> RR_calf -> RR_foot
+         -> imu_link
+         -> lidar_link
+         -> radar
+         -> front_camera_link
+  Topics/TF interface (unchanged):
+    /cmd_vel, /odom, /unilidar/cloud, /unilidar/imu
+    TF: odom -> base_footprint -> base_link
 -->
 <robot name="go2_sim" xmlns:xacro="http://www.ros.org/wiki/xacro">
-  <!-- ═══════════════════════════════════════════════════════════════════
-       sensor_models: reusable L1 LiDAR macro
-  ════════════════════════════════════════════════════════════════════════ -->
+  <!-- L1 LiDAR macro (unchanged) -->
   <xacro:include filename="$(find sensor_models)/urdf/l1_lidar.urdf.xacro"/>
-  <!-- ═══════════════════════════════════════════════════════════════════
-       Physical constants (source: root official go2.urdf in this repository)
-  ════════════════════════════════════════════════════════════════════════ -->
-  <xacro:property name="body_length"     value="0.3762"/>
-  <xacro:property name="body_width"      value="0.04675"/>   <!-- trunk half-width -->
-  <xacro:property name="body_height"     value="0.114"/>
-  <xacro:property name="body_mass"       value="6.921"/>
-  <xacro:property name="base_link_height_from_ground" value="0.335"/>
-  <!-- Front-top sensor mount from root official go2.urdf Head_upper_joint -->
-  <xacro:property name="lidar_x" value="0.285"/>
+  <!-- Physical constants (upstream go2_description const/urdf values) -->
+  <xacro:property name="trunk_length" value="0.3762"/>
+  <xacro:property name="trunk_width" value="0.0935"/>
+  <xacro:property name="trunk_height" value="0.114"/>
+  <xacro:property name="trunk_mass" value="6.921"/>
+  <!-- Standing pose -->
+  <xacro:property name="q_hip" value="0.0"/>
+  <xacro:property name="q_thigh" value="0.67"/>
+  <xacro:property name="q_calf" value="-1.30"/>
+  <!-- Base height in world when feet are on ground -->
+  <xacro:property name="base_z" value="0.380"/>
+  <!-- LiDAR mount from official Unitree Go2 specifications (radar_joint) -->
+  <xacro:property name="lidar_x" value="0.28945"/>
   <xacro:property name="lidar_y" value="0.0"/>
-  <xacro:property name="lidar_z" value="0.01"/>
-  <!-- ═══════════════════════════════════════════════════════════════════
-       base_footprint  —  ground-plane reference (Nav2 root)
-  ════════════════════════════════════════════════════════════════════════ -->
+  <xacro:property name="lidar_z" value="-0.046825"/>
+  <xacro:property name="lidar_r" value="0.0"/>
+  <!-- <xacro:property name="lidar_p" value="2.8782"/> -->
+  <xacro:property name="lidar_p" value="0.0"/>
+  <xacro:property name="lidar_yaw" value="0.0"/>
+  <!-- Mesh package (Option A: vendored meshes in go2_sim) -->
+  <xacro:property name="mesh_pkg" value="go2_sim"/>
   <link name="base_footprint">
-    <!-- Zero-size visual; Gazebo needs at least a tiny geometry for physics -->
     <visual>
       <geometry><box size="0.001 0.001 0.001"/></geometry>
     </visual>
-    <!-- No inertial on base_footprint; mass is in base_link -->
-  </link>
-  <!-- ═══════════════════════════════════════════════════════════════════
-       base_link  —  robot trunk centre
-  ════════════════════════════════════════════════════════════════════════ -->
+  </link>
   <joint name="base_footprint_to_base_link" type="fixed">
     <parent link="base_footprint"/>
-    <child  link="base_link"/>
-    <origin xyz="0 0 ${base_link_height_from_ground}" rpy="0 0 0"/>
+    <child link="base_link"/>
+    <origin xyz="0 0 ${base_z}" rpy="0 0 0"/>
   </joint>
   <link name="base_link">
-    <visual>
-      <origin xyz="0 0 0" rpy="0 0 0"/>
-      <geometry>
-        <box size="${body_length} ${body_width*2} ${body_height}"/>
-      </geometry>
-      <material name="dark_grey">
-        <color rgba="0.2 0.2 0.2 1.0"/>
-      </material>
-    </visual>
-    <collision>
-      <origin xyz="0 0 0" rpy="0 0 0"/>
-      <geometry>
-        <box size="${body_length} ${body_width*2} ${body_height}"/>
-      </geometry>
-    </collision>
-    <collision>
-      <!-- Contact proxy from official URDF zero-pose collision envelope; bottom at z=0 -->
-      <origin xyz="0 0 -0.325" rpy="0 0 0"/>
-      <geometry>
-        <box size="0.5794 0.328 0.020"/>
-      </geometry>
-    </collision>
-    <inertial>
-      <origin xyz="0.021112 0.0 -0.005366" rpy="0 0 0"/>
-      <mass value="${body_mass}"/>
-      <inertia ixx="0.02448"  ixy="0.00012166" ixz="0.0014849"
-               iyy="0.098077" iyz="-0.0000312"
-               izz="0.107"/>
-    </inertial>
-  </link>
-  <!-- ═══════════════════════════════════════════════════════════════════
-       imu_link  —  co-located with trunk centre
-  ════════════════════════════════════════════════════════════════════════ -->
-  <joint name="base_link_to_imu" type="fixed">
-    <parent link="base_link"/>
-    <child  link="imu_link"/>
-    <origin xyz="0 0 0" rpy="0 0 0"/>
+    <inertial>
+      <origin xyz="0.021112 0 -0.005366" rpy="0 0 0"/>
+      <mass value="${trunk_mass}"/>
+      <inertia ixx="0.02448" ixy="0.00012166" ixz="0.0014849" iyy="0.098077" iyz="-3.12E-05" izz="0.107"/>
+    </inertial>
+    <visual>
+      <origin xyz="0 0 0" rpy="0 0 0"/>
+      <geometry>
+        <mesh filename="package://${mesh_pkg}/meshes/dae/base.dae"/>
+      </geometry>
+    </visual>
+    <collision>
+      <origin rpy="0 0 0" xyz="0 0 0"/>
+      <geometry>
+        <box size="${trunk_length} ${trunk_width} ${trunk_height}"/>
+      </geometry>
+    </collision>
+  </link>
+  <link name="FL_hip">
+    <inertial>
+      <origin xyz="-0.0054 0.00194 -0.000105" rpy="0 0 0"/>
+      <mass value="0.678"/>
+      <inertia ixx="0.00048" ixy="-3.01E-06" ixz="1.11E-06" iyy="0.000884" iyz="-1.42E-06" izz="0.000596"/>
+    </inertial>
+    <visual>
+      <origin xyz="0 0 0" rpy="0 0 0"/>
+      <geometry>
+        <mesh filename="package://${mesh_pkg}/meshes/dae/hip.dae"/>
+      </geometry>
+    </visual>
+    <collision>
+      <origin rpy="1.5707963267948966 0 0" xyz="0 0.08 0"/>
+      <geometry>
+        <cylinder length="0.04" radius="0.046"/>
+      </geometry>
+    </collision>
+  </link>
+  <joint name="FL_hip_joint" type="fixed">
+    <origin xyz="0.1934 0.0465 0" rpy="${q_hip} 0 0"/>
+    <parent link="base_link"/>
+    <child link="FL_hip"/>
+  </joint>
+  <link name="FL_hip_rotor">
+    <inertial>
+      <origin rpy="0 0 0" xyz="0.0 0.0 0.0"/>
+      <mass value="0.089"/>
+      <inertia ixx="0.000111842" ixy="0.0" ixz="0.0" iyy="0.000059647" iyz="0.0" izz="0.000059647"/>
+    </inertial>
+  </link>
+  <joint name="FL_hip_rotor_joint" type="fixed">
+    <origin rpy="0 0 0" xyz="0.11215 0.04675 0"/>
+    <parent link="base_link"/>
+    <child link="FL_hip_rotor"/>
+  </joint>
+  <link name="FL_thigh">
+    <inertial>
+      <origin xyz="-0.00374 -0.0223 -0.0327" rpy="0 0 0"/>
+      <mass value="1.152"/>
+      <inertia ixx="0.00584" ixy="8.72E-05" ixz="-0.000289" iyy="0.0058" iyz="0.000808" izz="0.00103"/>
+    </inertial>
+    <visual>
+      <origin xyz="0 0 0" rpy="0 0 0"/>
+      <geometry>
+        <mesh filename="package://${mesh_pkg}/meshes/dae/thigh.dae"/>
+      </geometry>
+    </visual>
+    <collision>
+      <origin rpy="0 1.5707963267948966 0" xyz="0 0 -0.1065"/>
+      <geometry>
+        <box size="0.213 0.0245 0.034"/>
+      </geometry>
+    </collision>
+  </link>
+  <joint name="FL_thigh_joint" type="fixed">
+    <origin xyz="0 0.0955 0" rpy="0 ${q_thigh} 0"/>
+    <parent link="FL_hip"/>
+    <child link="FL_thigh"/>
+  </joint>
+  <link name="FL_thigh_rotor">
+    <inertial>
+      <origin rpy="0 0 0" xyz="0.0 0.0 0.0"/>
+      <mass value="0.089"/>
+      <inertia ixx="0.000059647" ixy="0.0" ixz="0.0" iyy="0.000111842" iyz="0.0" izz="0.000059647"/>
+    </inertial>
+  </link>
+  <joint name="FL_thigh_rotor_joint" type="fixed">
+    <origin rpy="0 0 0" xyz="0 -0.00015 0"/>
+    <parent link="FL_hip"/>
+    <child link="FL_thigh_rotor"/>
+  </joint>
+  <link name="FL_calf">
+    <inertial>
+      <origin xyz="0.00548 -0.000975 -0.115" rpy="0 0 0"/>
+      <mass value="0.154"/>
+      <inertia ixx="0.00108" ixy="3.4E-07" ixz="1.72E-05" iyy="0.0011" iyz="8.28E-06" izz="3.29E-05"/>
+    </inertial>
+    <visual>
+      <origin xyz="0 0 0" rpy="0 0 0"/>
+      <geometry>
+        <mesh filename="package://${mesh_pkg}/meshes/dae/calf.dae"/>
+      </geometry>
+    </visual>
+    <collision>
+      <origin rpy="0 -0.21 0" xyz="0.008 0 -0.06"/>
+      <geometry>
+        <cylinder length="0.12" radius="0.012"/>
+      </geometry>
+    </collision>
+  </link>
+  <joint name="FL_calf_joint" type="fixed">
+    <origin xyz="0 0 -0.213" rpy="0 ${q_calf} 0"/>
+    <parent link="FL_thigh"/>
+    <child link="FL_calf"/>
+  </joint>
+  <link name="FL_calflower">
+    <collision>
+      <origin rpy="0 0 0" xyz="0 0 0"/>
+      <geometry>
+        <cylinder length="0.065" radius="0.011"/>
+      </geometry>
+    </collision>
+  </link>
+  <joint name="FL_calflower_joint" type="fixed">
+    <origin xyz="0.020 0 -0.148" rpy="0 0.05 0"/>
+    <parent link="FL_calf"/>
+    <child link="FL_calflower"/>
+  </joint>
+  <link name="FL_calflower1">
+    <collision>
+      <origin rpy="0 0 0" xyz="0 0 0"/>
+      <geometry>
+        <cylinder length="0.03" radius="0.0155"/>
+      </geometry>
+    </collision>
+  </link>
+  <joint name="FL_calflower1_joint" type="fixed">
+    <origin xyz="-0.01 0 -0.04" rpy="0 0.48 0"/>
+    <parent link="FL_calflower"/>
+    <child link="FL_calflower1"/>
+  </joint>
+  <link name="FL_calf_rotor">
+    <inertial>
+      <origin rpy="0 0 0" xyz="0.0 0.0 0.0"/>
+      <mass value="0.089"/>
+      <inertia ixx="0.000059647" ixy="0.0" ixz="0.0" iyy="0.000111842" iyz="0.0" izz="0.000059647"/>
+    </inertial>
+  </link>
+  <joint name="FL_calf_rotor_joint" type="fixed">
+    <origin rpy="0 0 0" xyz="0 -0.03235 0"/>
+    <parent link="FL_thigh"/>
+    <child link="FL_calf_rotor"/>
+  </joint>
+  <link name="FL_foot">
+    <inertial>
+      <origin xyz="0 0 0" rpy="0 0 0"/>
+      <mass value="0.04"/>
+      <inertia ixx="9.6e-06" ixy="0" ixz="0" iyy="9.6e-06" iyz="0" izz="9.6e-06"/>
+    </inertial>
+    <visual>
+      <origin xyz="0 0 0" rpy="0 0 0"/>
+      <geometry>
+        <mesh filename="package://${mesh_pkg}/meshes/dae/foot.dae"/>
+      </geometry>
+    </visual>
+    <collision>
+      <origin rpy="0 0 0" xyz="-0.002 0 0"/>
+      <geometry>
+        <sphere radius="0.022"/>
+      </geometry>
+    </collision>
+  </link>
+  <joint name="FL_foot_joint" type="fixed">
+    <origin xyz="0 0 -0.213" rpy="0 0 0"/>
+    <parent link="FL_calf"/>
+    <child link="FL_foot"/>
+  </joint>
+  <link name="FR_hip">
+    <inertial>
+      <origin xyz="-0.0054 -0.00194 -0.000105" rpy="0 0 0"/>
+      <mass value="0.678"/>
+      <inertia ixx="0.00048" ixy="3.01E-06" ixz="1.11E-06" iyy="0.000884" iyz="1.42E-06" izz="0.000596"/>
+    </inertial>
+    <visual>
+      <origin xyz="0 0 0" rpy="3.1415 0 0"/>
+      <geometry>
+        <mesh filename="package://${mesh_pkg}/meshes/dae/hip.dae"/>
+      </geometry>
+    </visual>
+    <collision>
+      <origin rpy="1.5707963267948966 0 0" xyz="0 -0.08 0"/>
+      <geometry>
+        <cylinder length="0.04" radius="0.046"/>
+      </geometry>
+    </collision>
+  </link>
+  <joint name="FR_hip_joint" type="fixed">
+    <origin xyz="0.1934 -0.0465 0" rpy="${q_hip} 0 0"/>
+    <parent link="base_link"/>
+    <child link="FR_hip"/>
+  </joint>
+  <link name="FR_hip_rotor">
+    <inertial>
+      <origin rpy="0 0 0" xyz="0.0 0.0 0.0"/>
+      <mass value="0.089"/>
+      <inertia ixx="0.000111842" ixy="0.0" ixz="0.0" iyy="0.000059647" iyz="0.0" izz="0.000059647"/>
+    </inertial>
+  </link>
+  <joint name="FR_hip_rotor_joint" type="fixed">
+    <origin rpy="0 0 0" xyz="0.11215 -0.04675 0"/>
+    <parent link="base_link"/>
+    <child link="FR_hip_rotor"/>
+  </joint>
+  <link name="FR_thigh">
+    <inertial>
+      <origin xyz="-0.00374 0.0223 -0.0327" rpy="0 0 0"/>
+      <mass value="1.152"/>
+      <inertia ixx="0.00584" ixy="-8.72E-05" ixz="-0.000289" iyy="0.0058" iyz="-0.000808" izz="0.00103"/>
+    </inertial>
+    <visual>
+      <origin xyz="0 0 0" rpy="0 0 0"/>
+      <geometry>
+        <mesh filename="package://${mesh_pkg}/meshes/dae/thigh_mirror.dae"/>
+      </geometry>
+    </visual>
+    <collision>
+      <origin rpy="0 1.5707963267948966 0" xyz="0 0 -0.1065"/>
+      <geometry>
+        <box size="0.213 0.0245 0.034"/>
+      </geometry>
+    </collision>
+  </link>
+  <joint name="FR_thigh_joint" type="fixed">
+    <origin xyz="0 -0.0955 0" rpy="0 ${q_thigh} 0"/>
+    <parent link="FR_hip"/>
+    <child link="FR_thigh"/>
+  </joint>
+  <link name="FR_thigh_rotor">
+    <inertial>
+      <origin rpy="0 0 0" xyz="0.0 0.0 0.0"/>
+      <mass value="0.089"/>
+      <inertia ixx="0.000059647" ixy="0.0" ixz="0.0" iyy="0.000111842" iyz="0.0" izz="0.000059647"/>
+    </inertial>
+  </link>
+  <joint name="FR_thigh_rotor_joint" type="fixed">
+    <origin rpy="0 0 0" xyz="0 0.00015 0"/>
+    <parent link="FR_hip"/>
+    <child link="FR_thigh_rotor"/>
+  </joint>
+  <link name="FR_calf">
+    <inertial>
+      <origin xyz="0.00548 0.000975 -0.115" rpy="0 0 0"/>
+      <mass value="0.154"/>
+      <inertia ixx="0.00108" ixy="-3.4E-07" ixz="1.72E-05" iyy="0.0011" iyz="-8.28E-06" izz="3.29E-05"/>
+    </inertial>
+    <visual>
+      <origin xyz="0 0 0" rpy="0 0 0"/>
+      <geometry>
+        <mesh filename="package://${mesh_pkg}/meshes/dae/calf_mirror.dae"/>
+      </geometry>
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