Commit message: - Removed `sim_nav.launch.py` as it was redundant. - Updated `package.xml` to reflect changes in simulation description. - Modified `cloud_self_filter.py` to improve comments and adjust parameters. - Updated `l1_lidar.urdf.xacro` to correct topic names and remove legacy code. - Added `sim_classic_bringup.launch.py` for full Gazebo Classic simulation setup. - Added `topic_map.md` for authoritative reference on ROS 2 topics in the autonomy stack.

File: src/go2_description/urdf/go2.urdf.xacro (robot description, xacro)
@@ -14,6 +14,6 @@
     - Leg links are omitted (not needed for Nav2). Add them when joint-state
       visualization or IK is required.
-  TODO(sim): Add <gazebo> plugins block (LiDAR ray sensor, IMU sensor, skid-steer
-             or effort controller) behind an xacro:if use_gazebo argument.
+  NOTE: Gazebo simulation plugins are implemented in go2_sim/urdf/go2_sim.urdf.xacro.
+        This hardware-focused URDF intentionally keeps simulation plugins out.
   TODO(agibot): Create agibot_d1_description/urdf/d1.urdf.xacro with the same
                 frame names (base_footprint, base_link, lidar_link, imu_link).
@@ -45,5 +45,4 @@
   <xacro:property name="lidar_z" value="-0.046825"/>
   <xacro:property name="lidar_r" value="0.0"/>
-  <!-- <xacro:property name="lidar_p" value="2.8782"/> -->
   <xacro:property name="lidar_p" value="0.0"/>
   <xacro:property name="lidar_yaw" value="0.0"/>
@@ -171,5 +170,5 @@
   <!-- ═══════════════════════════════════════════════════════════════════════
        Gazebo plugins  (only included when use_gazebo:=true)
-       TODO(sim): Replace stubs with working Gazebo Humble plugins.
+       NOTE: these placeholders remain intentionally empty in this hardware URDF.
   ════════════════════════════════════════════════════════════════════════════ -->
   <xacro:if value="$(arg use_gazebo)">
@@ -178,7 +177,5 @@
       <material>Gazebo/DarkGrey</material>
     </gazebo>
-    <!-- TODO(sim): Add Gazebo LiDAR ray plugin on lidar_link -->
-    <!-- TODO(sim): Add Gazebo IMU plugin on imu_link -->
-    <!-- TODO(sim): Add differential-drive or effort controller plugin -->
+    <!-- Simulation plugins are provided by go2_sim/urdf/go2_sim.urdf.xacro -->
   </xacro:if>
 </robot>

File: src/go2_sim/urdf/go2_sim.urdf.xacro (robot description, xacro)
@@ -80,5 +80,4 @@
   <!-- ════════════════════════════════════════════════════════════════════
        TRUNK  (main body visual / collision / inertia)
-       Mesh: base.dae  (byte-identical to source trunk.dae; same 10727399 B)
        ════════════════════════════════════════════════════════════════════ -->
   <joint name="floating_base" type="fixed">
@@ -237,5 +236,5 @@
          xyz = (0.28945, 0, -0.046825) relative to base_link
        The macro creates lidar_link (with prefix="") and publishes on
-       Ignition topic /unilidar/cloud/points, bridged to ROS /lidar/points.
+       Ignition topic /lidar/points, bridged to ROS /lidar/points.
        Frame "lidar_link" matches:
          scan_from_cloud.yaml  target_frame: lidar_link
@@ -244,5 +243,5 @@
        ════════════════════════════════════════════════════════════════════ -->
   <xacro:l1_lidar parent="base_link" prefix="">
-    <origin xyz="0.28945 0 -0.046825" rpy="0 2.8782 0"/>
+    <origin xyz="0.28945 0 -0.046825" rpy="0 0 0"/>
   </xacro:l1_lidar>
 </robot>

File: src/sensor_models/urdf/l1_lidar.urdf.xacro (robot description, xacro)
@@ -31,7 +31,6 @@
     - Joint: ${prefix}lidar_l1_joint  (fixed, parent→child, origin from block)
     - Gazebo gpu_lidar sensor on ${prefix}lidar_link
-      Gazebo topics:
-        /unilidar/cloud         (LaserScan)
-        /unilidar/cloud/points  (PointCloudPacked, bridged to ROS /lidar/points)
+      Gazebo topic:
+        /lidar/points  (PointCloudPacked, bridged to ROS /lidar/points)
   ─────────────────────────────────────────────────────────────────────────────
   MACRO: l1_lidar_gazebo  (Classic / Gazebo 11) — legacy, do not use for Fortress
@@ -47,5 +46,5 @@
       parent
       prefix
-      range_min:=0.8
+      range_min:=0.1
       range_max:=30.0
       *origin">
@@ -79,10 +78,9 @@
       With prefix="" this yields "lidar_link" which matches scan_from_cloud.yaml
       (target_frame: lidar_link) and go2_description/go2_bringup conventions.
-      PointCloud topic /unilidar/cloud/points is bridged by ros_ign_bridge
-      in the launch file to ROS topic /lidar/points.
+      PointCloud topic /lidar/points is bridged by ros_ign_bridge in the launch file.
     -->
     <gazebo reference="${prefix}lidar_link">
       <sensor name="${prefix}lidar_l1" type="gpu_lidar">
-        <topic>/unilidar/cloud</topic>
+        <topic>/lidar/points</topic>
         <update_rate>10</update_rate>
         <always_on>1</always_on>
@@ -120,64 +118,3 @@
     </gazebo>
   </xacro:macro>
-  <!-- ═══════════════════════════════════════════════════════════════════════
-       CLASSIC MACRO  (Gazebo 11 / libgazebo_ros_ray_sensor)
-       Kept for the robot_sim Gazebo Classic pipeline.  Do NOT use in Fortress.
-       ═══════════════════════════════════════════════════════════════════════ -->
-  <xacro:macro name="l1_lidar_gazebo" params="
-      parent_link
-      topic:='/lidar/points'
-      update_rate:=10
-      h_samples:=360
-      v_samples:=18
-      v_min_angle_deg:=-45.0
-      v_max_angle_deg:=45.0
-      range_min:=0.15
-      range_max:=30.0
-      noise_stddev:=0.02
-      visualize:=false
-  ">
-    <xacro:property name="deg_to_rad" value="${pi / 180.0}"/>
-    <xacro:property name="v_min_rad"  value="${v_min_angle_deg * deg_to_rad}"/>
-    <xacro:property name="v_max_rad"  value="${v_max_angle_deg * deg_to_rad}"/>
-    <gazebo reference="${parent_link}">
-      <sensor type="gpu_ray" name="l1_lidar">
-        <pose>0 0 0 0 0 0</pose>
-        <visualize>${visualize}</visualize>
-        <update_rate>${update_rate}</update_rate>
-        <ray>
-          <scan>
-            <horizontal>
-              <samples>${h_samples}</samples>
-              <resolution>1</resolution>
-              <min_angle>-3.14159265358979</min_angle>
-              <max_angle> 3.14159265358979</max_angle>
-            </horizontal>
-            <vertical>
-              <samples>${v_samples}</samples>
-              <resolution>1</resolution>
-              <min_angle>${v_min_rad}</min_angle>
-              <max_angle>${v_max_rad}</max_angle>
-            </vertical>
-          </scan>
-          <range>
-            <min>${range_min}</min>
-            <max>${range_max}</max>
-            <resolution>0.001</resolution>
-          </range>
-          <noise>
-            <type>gaussian</type>
-            <mean>0.0</mean>
-            <stddev>${noise_stddev}</stddev>
-          </noise>
-        </ray>
-        <plugin name="gazebo_ros_l1_lidar" filename="libgazebo_ros_ray_sensor.so">
-          <ros>
-            <remapping>~/out:=${topic}</remapping>
-          </ros>
-          <output_type>sensor_msgs/PointCloud2</output_type>
-          <frame_name>${parent_link}</frame_name>
-        </plugin>
-      </sensor>
-    </gazebo>
-  </xacro:macro>
 </robot>

Commit message: Refactor navigation and sensor configurations for Unitree Go2
- Updated `ros_control.yaml` to include `ff_velocity_scale` for joint gains to avoid deprecation warnings.
- Modified `sim_champ.launch.py` to remap LiDAR topics and clarify TF bridging notes to prevent cycles in the TF tree.
- Enhanced `nav2_params.yaml` with new parameters for the SmacPlanner and adjusted penalties for better navigation performance.
- Adjusted `nav2_params_2d.yaml` to include similar updates as `nav2_params.yaml`.
- Added a warning in `ekf.launch.py` to prevent conflicts when launching EKF alongside simulation launches.
- Updated `l1_lidar.urdf.xacro` to reflect changes in LiDAR topic names and clarify sensor configurations.
- Introduced `nav_realrobot.launch.py` for launching the navigation stack on real robots, ensuring compatibility with existing hardware setups.

File: src/go2_description/urdf/go2.urdf.xacro (robot description, xacro)
@@ -20,8 +20,4 @@
 -->
 <robot name="go2" xmlns:xacro="http://www.ros.org/wiki/xacro">
-  <!-- ═══════════════════════════════════════════════════════════════════════
-       Arguments
-  ════════════════════════════════════════════════════════════════════════════ -->
-  <xacro:arg name="use_gazebo" default="false"/>
   <!-- ═══════════════════════════════════════════════════════════════════════
        Physical constants
@@ -168,14 +164,6 @@
     </inertial>
   </link>
-  <!-- ═══════════════════════════════════════════════════════════════════════
-       Gazebo plugins  (only included when use_gazebo:=true)
-       NOTE: these placeholders remain intentionally empty in this hardware URDF.
-  ════════════════════════════════════════════════════════════════════════════ -->
-  <xacro:if value="$(arg use_gazebo)">
-    <!-- Gazebo material -->
-    <gazebo reference="base_link">
-      <material>Gazebo/DarkGrey</material>
-    </gazebo>
-    <!-- Simulation plugins are provided by go2_sim/urdf/go2_sim.urdf.xacro -->
-  </xacro:if>
+  <!-- FIX(agent5): Removed <gazebo> block that was present in go2_description.
+       All Gazebo material/plugin tags belong exclusively in go2_sim/urdf/go2_sim.urdf.xacro.
+       The use_gazebo xacro:arg is also removed as it is no longer referenced. -->
 </robot>

File: src/sensor_models/urdf/l1_lidar.urdf.xacro (robot description, xacro)
@@ -32,6 +32,6 @@
     - Gazebo gpu_lidar sensor on ${prefix}lidar_link
       Gazebo topics:
-        /lidar        (LaserScan — unused by nav stack)
-        /lidar/points (PointCloudPacked, bridged to ROS /lidar/points)
+        /unilidar/cloud        (LaserScan — unused by nav stack)
+        /unilidar/cloud/points (PointCloudPacked, bridged to ROS /lidar/points via remapping)
   ─────────────────────────────────────────────────────────────────────────────
   MACRO: l1_lidar_gazebo  (Classic / Gazebo 11) — legacy, do not use for Fortress
@@ -79,12 +79,14 @@
       With prefix="" this yields "lidar_link" which matches scan_from_cloud.yaml
       (target_frame: lidar_link) and go2_description/go2_bringup conventions.
-      PointCloud topic /lidar/points is bridged by ros_ign_bridge in the launch file.
+      PointCloud topic /unilidar/cloud/points is bridged and remapped to /lidar/points
+      by ros_ign_bridge in the launch file.
     -->
     <gazebo reference="${prefix}lidar_link">
       <sensor name="${prefix}lidar_l1" type="gpu_lidar">
-        <!-- gpu_lidar publishes PointCloudPacked on <topic>/points, so the base
-             topic must be /lidar to land the point cloud on /lidar/points (bridged
-             to ROS).  LaserScan lands on /lidar (unused by nav stack). -->
-        <topic>/lidar</topic>
+        <!-- FIX(agent1): sensor topic changed to /unilidar/cloud so gpu_lidar emits
+             /unilidar/cloud/points (PointCloudPacked).  The bridge in sim_champ.launch.py
+             bridges /unilidar/cloud/points and remaps it to the ROS topic /lidar/points.
+             This matches the Unitree L1 real-hardware topic name convention. -->
+        <topic>/unilidar/cloud</topic>
         <update_rate>10</update_rate>
         <always_on>1</always_on>

Commit message: - Add distortion corrector for LiDAR point clouds - Tune obstacle detection parameters

File: src/go2_description/urdf/go2.urdf.xacro (robot description, xacro)
@@ -4,11 +4,13 @@
   Minimal Go2 robot description for Nav2 navigation.
   Frame tree (Nav2 standard contract):
-    base_footprint  (ground projection, z=0 at foot contact level)
-      └─ base_link        (robot body center at standing height)
+    base_footprint  (published dynamically by the hardware bridge / sim launch)
+      └─ base_link        (robot body center at standing height, roll/pitch-capable)
            ├─ trunk        (visual/collision body mesh)
            ├─ imu_link     (co-located with trunk centre)
            └─ lidar_link   (Unitree L1 LiDAR mount)
   Notes:
-    - base_link is placed at nominal standing torso centre height (0.28 m above ground).
+    - This URDF is rooted at base_link. base_footprint is intentionally not part of
+      robot_description so bringup can publish base_footprint→base_link dynamically
+      from IMU roll/pitch without conflicting with robot_state_publisher.
     - lidar_link pose matches Go2 mounting location used by Nav2/SLAM.
     - Leg links are omitted (not needed for Nav2). Add them when joint-state
@@ -30,4 +32,6 @@
   <xacro:property name="stance_length"  value="0.700"/>  <!-- full X with legs -->
   <xacro:property name="stance_width"   value="0.310"/>  <!-- full Y with legs -->
+  <xacro:property name="safety_length"  value="0.800"/>  <!-- +50 mm safety margin on each side -->
+  <xacro:property name="safety_width"   value="0.410"/>  <!-- +50 mm safety margin on each side -->
   <xacro:property name="stance_height"  value="0.230"/>  <!-- approx clearance:
                                                               ground to body bottom
@@ -44,19 +48,6 @@
   <xacro:property name="lidar_yaw" value="0.0"/>
   <!-- ═══════════════════════════════════════════════════════════════════════
-       base_footprint  —  ground contact reference (Nav2 global frame anchor)
-  ════════════════════════════════════════════════════════════════════════════ -->
-  <link name="base_footprint">
-    <visual>
-      <geometry><box size="0.001 0.001 0.001"/></geometry>
-    </visual>
-  </link>
-  <!-- ═══════════════════════════════════════════════════════════════════════
        base_link  —  robot body centre
   ════════════════════════════════════════════════════════════════════════════ -->
-  <joint name="base_footprint_to_base_link" type="fixed">
-    <parent link="base_footprint"/>
-    <child  link="base_link"/>
-    <origin xyz="0 0 ${standing_height}" rpy="0 0 0"/>
-  </joint>
   <link name="base_link">
     <visual>
@@ -76,5 +67,5 @@
       </material>
     </visual>
-    <!-- Leg stance envelope — represents full swept area including legs.
+    <!-- Leg stance envelope — represents the physical standing footprint.
          Positioned at z = -(standing_height - stance_height/2) relative to
          base_link, which is: -(0.28 - 0.115) = -0.165 m -->
@@ -101,11 +92,9 @@
       </geometry>
     </collision>
-    <!-- Leg stance envelope — represents full swept area including legs.
-         Positioned at z = -(standing_height - stance_height/2) relative to
-         base_link, which is: -(0.28 - 0.115) = -0.165 m -->
+    <!-- Safety envelope used by collision consumers that inspect URDF collision geometry. -->
     <collision>
       <origin xyz="0 0 ${-(standing_height - stance_height/2)}" rpy="0 0 0"/>
       <geometry>
-        <box size="${stance_length} ${stance_width} ${stance_height}"/>
+        <box size="${safety_length} ${safety_width} ${stance_height}"/>
       </geometry>
     </collision>

File: src/go2_sim/urdf/go2_sim.urdf.xacro (robot description, xacro)
@@ -255,5 +255,7 @@
        ════════════════════════════════════════════════════════════════════ -->
   <xacro:l1_lidar parent="base_link" prefix="">
-    <origin xyz="0.28945 0 -0.046825" rpy="0 0 0"/>
+    <!-- The Unitree L1 is mounted upside down on Go2, so its upward
+         hemispherical scan in sensor frame points toward the floor. -->
+    <origin xyz="0.28945 0 -0.056825" rpy="3.14159265358979 0 0"/>
   </xacro:l1_lidar>
 </robot>

File: src/sensor_models/urdf/l1_lidar.urdf.xacro (robot description, xacro)
@@ -10,6 +10,6 @@
   ─────────────────────────────────────────────────────────────────────────────
   Unitree L1 device specifications (from Unitree datasheet):
-    - Scan lines (vertical channels): 18 (simulation uses 30 for fidelity)
-    - Vertical FOV: ±45° (−45° to +45°)
+    - Scan lines (vertical channels): 18 (simulation uses 32 for fidelity)
+    - Vertical FOV: 90° hemispherical
     - Horizontal FOV: 360°
     - Rotation frequency (typical): 10 Hz
@@ -34,9 +34,4 @@
         /unilidar/cloud        (LaserScan — unused by nav stack)
         /unilidar/cloud/points (PointCloudPacked, bridged to ROS /lidar/points via remapping)
-  ─────────────────────────────────────────────────────────────────────────────
-  MACRO: l1_lidar_gazebo  (Classic / Gazebo 11) — legacy, do not use for Fortress
-  ─────────────────────────────────────────────────────────────────────────────
-  Usage:
-    <xacro:l1_lidar_gazebo parent_link="lidar_link"/>
 -->
 <robot xmlns:xacro="http://www.ros.org/wiki/xacro">
@@ -47,5 +42,5 @@
       parent
       prefix
-      range_min:=0.05
+      range_min:=0.1
       range_max:=30.0
       *origin">
@@ -84,38 +79,32 @@
     <gazebo reference="${prefix}lidar_link">
       <sensor name="${prefix}lidar_l1" type="gpu_lidar">
-        <!-- FIX(agent1): sensor topic changed to /unilidar/cloud so gpu_lidar emits
-             /unilidar/cloud/points (PointCloudPacked).  The bridge in sim_champ.launch.py
-             bridges /unilidar/cloud/points and remaps it to the ROS topic /lidar/points.
-             This matches the Unitree L1 real-hardware topic name convention. -->
         <topic>/unilidar/cloud</topic>
-        <update_rate>10</update_rate>
-        <always_on>1</always_on>
-        <!-- <visualize>false</visualize> -->
+        <update_rate>11</update_rate>
+        <always_on>true</always_on>
+        <visualize>true</visualize>
         <ignition_frame_id>${prefix}lidar_link</ignition_frame_id>
-        <!-- Ignition Fortress gpu_lidar requires <lidar>, not <ray> (Gazebo Classic).
-             Using <ray> causes Ignition to ignore the config and fall back to a
-             narrow default FOV, producing only a front-arc partial scan. -->
         <lidar>
           <scan>
             <horizontal>
               <!-- 360° sweep — L1 spec: 360° horizontal FOV -->
-              <samples>600</samples>
+              <samples>360</samples>
               <resolution>1</resolution>
-              <min_angle>-3.14159265358979</min_angle>
+              <min_angle>-3.14159265358978</min_angle>
               <max_angle>3.14159265358979</max_angle>
             </horizontal>
             <vertical>
-              <!-- ±45° vertical FOV — L1 spec: 90° vertical FOV (±45°) -->
-              <samples>30</samples>
+              <!-- 90° hemisphere in sensor frame; the Go2 mount flips the sensor
+                   so this sweeps toward the floor in the world frame. -->
+              <samples>32</samples>
               <resolution>1</resolution>
-              <min_angle>-0.78539816339745</min_angle>
-              <max_angle>0.78539816339745</max_angle>
+              <min_angle>0.00</min_angle>
+              <max_angle>1.5</max_angle>
             </vertical>
           </scan>
           <range>
-            <!-- L1 spec: 0.05 m min, 30 m max (L1 RM variant) -->
+            <!-- Fortress is stable here with a 0.1 m near clip. -->
             <min>${range_min}</min>
             <max>${range_max}</max>
-            <resolution>0.001</resolution>
+            <resolution>0.01</resolution>
           </range>
           <noise>

Commit message: Enhance SLAM and PointCloud Processing for Improved Navigation
- Updated scan_from_cloud.yaml to use a stabilized lidar frame, adjusted height filters, and refined angular scan parameters for better scan density.
- Modified slam_toolbox_params.yaml to increase motion thresholds and reduce maximum laser range for improved stability in indoor environments.
- Enhanced slam.launch.py to include new parameters for scan processing and distortion correction, allowing for more flexible configurations.
- Improved distortion_corrector.py to support a bypass mode for simulation scenarios, ensuring accurate point cloud processing.
- Added cloud_self_filter.py to mask robot-body and below-floor returns from point clouds, improving navigation accuracy.
- Updated URDF for lidar to prevent self-occlusion in simulation.
- Created new indoor_office.world and modified existing worlds to include necessary plugins for sensor integration and physics.
- Added scripts for managing ROS nodes and running the GO2 robot in both real and simulation environments.

File: src/go2_description/urdf/go2.urdf.xacro (robot description, xacro)
@@ -141,10 +141,4 @@
       </material>
     </visual>
-    <collision>
-      <origin xyz="0 0 0" rpy="0 0 0"/>
-      <geometry>
-        <cylinder radius="0.04" length="0.06"/>
-      </geometry>
-    </collision>
     <inertial>
       <mass value="0.001"/>

File: src/sensor_models/urdf/l1_lidar.urdf.xacro (robot description, xacro)
@@ -46,13 +46,5 @@
       *origin">
     <link name="${prefix}lidar_link">
-      <visual>
-        <origin xyz="0 0 0" rpy="0 0 0"/>
-        <geometry>
-          <cylinder radius="0.04" length="0.05"/>
-        </geometry>
-        <material name="lidar_black">
-          <color rgba="0.05 0.05 0.05 1.0"/>
-        </material>
-      </visual>
+      <!-- No visual geometry in sim: prevents GPU LiDAR self-occlusion at the sensor origin. -->
       <inertial>
         <mass value="0.5"/>
