Commit message: Refactor simulation files for Gazebo Fortress compatibility and remove legacy support

File: src/d1_sim/urdf/d1_sim.urdf.xacro (robot description, xacro)
@@ -2,5 +2,5 @@
 <!--
   d1_sim.urdf.xacro
-  AgiBot D1 Ultra — Gazebo Classic (Gazebo 11) simulation model STUB.
+  AgiBot D1 Ultra — Gazebo Fortress simulation model STUB.
   TODO(agibot): Implement this file following go2_sim/urdf/go2_sim.urdf.xacro as a template.
   Checklist:
@@ -8,13 +8,12 @@
     [ ] 2. Update standing_height, lidar_x/y/z to D1 Ultra geometry
     [ ] 3. Choose sensor macro:
-            Option A — reuse l1_lidar_gazebo with D1's LiDAR parameters
-            Option B — add a d1_lidar_gazebo macro to sensor_models/ if D1 uses a different LiDAR
-    [ ] 4. Keep the libgazebo_ros_planar_move block UNCHANGED (same topics, same frames)
-    [ ] 5. Keep frame names UNCHANGED: base_footprint, base_link, lidar_link, imu_link
-    [ ] 6. Update robot_name attribute to "d1_ultra"
+        Option A — reuse l1_lidar with D1's LiDAR parameters
+        Option B — add a d1_lidar macro to sensor_models/ if D1 uses a different LiDAR
+      [ ] 4. Keep frame names UNCHANGED: base_footprint, base_link, lidar_link, imu_link
+      [ ] 5. Update robot_name attribute to "d1_ultra"
   After implementing, launch with:
     ros2 launch robot_sim sim_bringup.launch.py robot:=d1
 -->
-<robot name="d1_ultra_STUB" xmlns:xacro="http://www.ros.org/wiki/xacro">
+<robot name="d1_ultra_stub" xmlns:xacro="http://www.ros.org/wiki/xacro">
   <xacro:include filename="$(find sensor_models)/urdf/l1_lidar.urdf.xacro"/>
   <!-- TODO(agibot): Replace with D1 Ultra physical specs -->
@@ -61,53 +60,14 @@
     </inertial>
   </link>
-  <joint name="base_link_to_lidar" type="fixed">
-    <parent link="base_link"/>
-    <child  link="lidar_link"/>
+  <!-- TODO(agibot): Update sensor params to D1 LiDAR specs if different from L1 -->
+  <xacro:l1_lidar parent="base_link" prefix="">
     <origin xyz="${lidar_x} ${lidar_y} ${lidar_z}" rpy="0 0 0"/>
-  </joint>
-  <link name="lidar_link">
-    <visual>
-      <geometry><cylinder radius="0.04" length="0.06"/></geometry>
-      <material name="lidar_black"><color rgba="0.05 0.05 0.05 1.0"/></material>
-    </visual>
-    <collision>
-      <geometry><cylinder radius="0.04" length="0.06"/></geometry>
-    </collision>
-    <inertial>
-      <mass value="0.3"/>
-      <origin xyz="0 0 0" rpy="0 0 0"/>
-      <inertia ixx="5e-4" ixy="0" ixz="0" iyy="5e-4" iyz="0" izz="5e-4"/>
-    </inertial>
-  </link>
-  <!-- Planar move plugin — DO NOT CHANGE (same interface as go2_sim) -->
-  <gazebo>
-    <plugin name="gazebo_ros_planar_move" filename="libgazebo_ros_planar_move.so">
-      <ros>
-        <remapping>cmd_vel:=/cmd_vel</remapping>
-        <remapping>odom:=/odom</remapping>
-      </ros>
-      <update_rate>50</update_rate>
-      <publish_odom>true</publish_odom>
-      <publish_odom_tf>true</publish_odom_tf>
-      <odometry_frame>odom</odometry_frame>
-      <robot_base_frame>base_footprint</robot_base_frame>
-      <covariance_x>0.0001</covariance_x>
-      <covariance_y>0.0001</covariance_y>
-      <covariance_yaw>0.01</covariance_yaw>
-    </plugin>
-  </gazebo>
-  <!-- TODO(agibot): Update sensor params to D1 LiDAR specs if different from L1 -->
-  <xacro:l1_lidar_gazebo
-      parent_link="lidar_link"
-      topic="/unilidar/cloud"
-  />
+  </xacro:l1_lidar>
   <gazebo reference="imu_link">
-    <sensor type="imu" name="d1_imu">
-      <always_on>true</always_on>
-      <update_rate>250</update_rate>
-      <plugin name="gazebo_ros_imu" filename="libgazebo_ros_imu_sensor.so">
-        <ros><remapping>~/out:=/unilidar/imu</remapping></ros>
-        <initial_orientation_as_reference>false</initial_orientation_as_reference>
-      </plugin>
+    <sensor name="d1_imu_sensor" type="imu">
+      <always_on>1</always_on>
+      <update_rate>200</update_rate>
+      <topic>/imu/data</topic>
+      <ignition_frame_id>imu_link</ignition_frame_id>
     </sensor>
   </gazebo>

File: src/go2_sim/urdf/go2_sim.urdf.xacro (robot description, xacro)
@@ -16,5 +16,5 @@
   CHAMP requires four foot links named exactly: LF_FOOT RF_FOOT LH_FOOT RH_FOOT
   These are generated by the leg macro in leg.xacro.
-  Fortress plugins used (all Classic libgazebo_ros_* plugins removed):
+  Fortress plugins used:
     - ign_ros2_control-system          (joint trajectory effort control)
     - ignition-gazebo-imu-system       (IMU sensor)
@@ -28,5 +28,4 @@
     /cmd_vel            — geometry_msgs/Twist        (ROS → Gazebo)
     /model/go2/odometry — nav_msgs/Odometry          (Ignition → ROS as /odom/raw → EKF)
-  DO NOT USE libgazebo_ros_* plugins here — they are Gazebo Classic only.
   DO NOT USE gz:: namespaces — Fortress uses ignition:: exclusively.
 -->

File: src/sensor_models/urdf/l1_lidar.urdf.xacro (robot description, xacro)
@@ -3,7 +3,6 @@
   l1_lidar.urdf.xacro
   Reusable sensor macros for the Unitree L1 LiDAR sensor.
-  Two macros are provided:
-    1. l1_lidar          — Gazebo Fortress (Ignition Gazebo 6, ROS 2 Humble) — USE THIS
-    2. l1_lidar_gazebo   — Gazebo Classic (Gazebo 11) — kept for robot_sim Classic pipeline
+  Macro provided:
+    1. l1_lidar          — Gazebo Fortress (Ignition Gazebo 6, ROS 2 Humble)
   ─────────────────────────────────────────────────────────────────────────────
   MACRO: l1_lidar  (Fortress / Ignition Gazebo 6)
