Commit message: docs: aligned with current code, cleaned up comments

File: src/simulation/d1_sim/urdf/d1_sim.urdf.xacro (robot description, xacro)
@@ -1,15 +1,11 @@
 <?xml version="1.0"?>
 <!--
-  d1_sim.urdf.xacro
-  AgiBot D1 Ultra — Gazebo Fortress simulation model STUB.
-  TODO(agibot): Implement this file following go2_sim/urdf/go2_sim.urdf.xacro as a template.
-  Checklist:
-    [ ] 1. Update physical constants (trunk dimensions, mass, inertia) to D1 Ultra datasheet values
-    [ ] 2. Update standing_height, lidar_x/y/z to D1 Ultra geometry
-    [ ] 3. Choose sensor macro:
-        Option A — reuse l1_lidar with D1's LiDAR parameters
-        Option B — add a d1_lidar macro to sensor_models/ if D1 uses a different LiDAR
-      [ ] 4. Keep frame names UNCHANGED: base_footprint, base_link, lidar_link, imu_link
-      [ ] 5. Update robot_name attribute to "d1_ultra"
+  d1_sim.urdf.xacro -- AgiBot D1 Ultra Gazebo Fortress simulation model STUB.
+  TODO(d1): Implement following go2_sim/urdf/go2_sim.urdf.xacro as template.
+    [ ] Update physical constants (trunk dimensions, mass, inertia) from D1 Ultra datasheet
+    [ ] Update standing_height, lidar_x/y/z to D1 Ultra geometry
+    [ ] Choose sensor: reuse l1_lidar macro or add a new one in sensor_models/ if needed
+    [ ] Keep frame names unchanged: base_footprint, base_link, lidar_link, imu_link
+    [ ] Update robot name attribute to "d1_ultra"
   After implementing, launch with:
     ros2 launch robot_sim sim_bringup.launch.py robot:=d1
@@ -17,6 +13,6 @@
 <robot name="d1_ultra_stub" xmlns:xacro="http://www.ros.org/wiki/xacro">
   <xacro:include filename="$(find sensor_models)/urdf/l1_lidar.urdf.xacro"/>
-  <!-- TODO(agibot): Replace with D1 Ultra physical specs -->
-  <xacro:property name="body_length"     value="0.50"/>   <!-- placeholder -->
+  <!-- TODO(d1): Replace with D1 Ultra physical specs -->
+  <xacro:property name="body_length"     value="0.50"/>
   <xacro:property name="body_width"      value="0.15"/>
   <xacro:property name="body_height"     value="0.12"/>
@@ -26,5 +22,4 @@
   <xacro:property name="lidar_y"         value="0.0"/>
   <xacro:property name="lidar_z"         value="0.20"/>
-  <!-- Frame tree (must match this exactly — no changes allowed) -->
   <link name="base_footprint">
     <visual><geometry><box size="0.001 0.001 0.001"/></geometry></visual>
@@ -44,5 +39,5 @@
     </collision>
     <inertial>
-      <!-- TODO(agibot): Replace with real D1 Ultra inertia tensor -->
+      <!-- TODO(d1): Replace with real D1 Ultra inertia tensor -->
       <origin xyz="0 0 0" rpy="0 0 0"/>
       <mass value="${body_mass}"/>
@@ -60,5 +55,5 @@
     </inertial>
   </link>
-  <!-- TODO(agibot): Update sensor params to D1 LiDAR specs if different from L1 -->
+  <!-- TODO(d1): Update sensor params to D1 LiDAR specs if different from L1 -->
   <xacro:l1_lidar parent="base_link" prefix="">
     <origin xyz="${lidar_x} ${lidar_y} ${lidar_z}" rpy="0 0 0"/>

File: src/simulation/go2_sim/urdf/go2_sim.urdf.xacro (robot description, xacro)
@@ -37,4 +37,14 @@
   <xacro:arg name="robot_controllers"
              default="$(find go2_sim)/config/ros_control.yaml"/>
+  <!-- Real lidar IMU calibration imported from imu_calib_data.yaml -->
+  <xacro:property name="lidar_imu_acc_bias_x" value="-0.801651"/>
+  <xacro:property name="lidar_imu_acc_bias_y" value="1.72345"/>
+  <xacro:property name="lidar_imu_acc_bias_z" value="-0.22166"/>
+  <xacro:property name="lidar_imu_ang_bias_x" value="0.00149071"/>
+  <xacro:property name="lidar_imu_ang_bias_y" value="0.00388548"/>
+  <xacro:property name="lidar_imu_ang_bias_z" value="0.00161095"/>
+  <!-- Derived from ang_z2x_proj=0.143694 and ang_z2y_proj=-0.19373 -->
+  <xacro:property name="lidar_imu_roll" value="0.194961"/>
+  <xacro:property name="lidar_imu_pitch" value="0.144193"/>
   <!-- == Include sub-files == -->
   <xacro:include filename="$(find go2_sim)/urdf/const.xacro"/>
@@ -269,5 +279,5 @@
     <parent link="lidar_link"/>
     <child  link="lidar_imu_link"/>
-    <origin xyz="-0.007698 -0.014655 0.00667" rpy="0 0 0"/>
+    <origin xyz="-0.007698 -0.014655 0.00667" rpy="${lidar_imu_roll} ${lidar_imu_pitch} 0"/>
   </joint>
   <link name="lidar_imu_link">
@@ -299,12 +309,12 @@
       <imu>
         <angular_velocity>
-          <x><noise type="gaussian"><mean>0</mean><stddev>0.009</stddev></noise></x>
-          <y><noise type="gaussian"><mean>0</mean><stddev>0.009</stddev></noise></y>
-          <z><noise type="gaussian"><mean>0</mean><stddev>0.009</stddev></noise></z>
+          <x><noise type="gaussian"><mean>${lidar_imu_ang_bias_x}</mean><stddev>0.009</stddev></noise></x>
+          <y><noise type="gaussian"><mean>${lidar_imu_ang_bias_y}</mean><stddev>0.009</stddev></noise></y>
+          <z><noise type="gaussian"><mean>${lidar_imu_ang_bias_z}</mean><stddev>0.009</stddev></noise></z>
         </angular_velocity>
         <linear_acceleration>
-          <x><noise type="gaussian"><mean>0</mean><stddev>0.021</stddev></noise></x>
-          <y><noise type="gaussian"><mean>0</mean><stddev>0.021</stddev></noise></y>
-          <z><noise type="gaussian"><mean>0</mean><stddev>0.021</stddev></noise></z>
+          <x><noise type="gaussian"><mean>${lidar_imu_acc_bias_x}</mean><stddev>0.021</stddev></noise></x>
+          <y><noise type="gaussian"><mean>${lidar_imu_acc_bias_y}</mean><stddev>0.021</stddev></noise></y>
+          <z><noise type="gaussian"><mean>${lidar_imu_acc_bias_z}</mean><stddev>0.021</stddev></noise></z>
         </linear_acceleration>
       </imu>

File: src/simulation/sensor_models/urdf/l1_lidar.urdf.xacro (robot description, xacro)
@@ -54,4 +54,10 @@
         </material>
       </visual>
+      <collision>
+        <origin xyz="0 0 0" rpy="0 0 0"/>
+        <geometry>
+          <cylinder radius="0.04" length="0.02"/>
+        </geometry>
+      </collision>
       <inertial>
         <mass value="0.5"/>
