Commit message: DLIO and EKF tuning for better odometry estimation

File: src/simulation/go2_sim/urdf/go2_sim.urdf.xacro (robot description, xacro)
@@ -279,5 +279,9 @@
     <parent link="lidar_link"/>
     <child  link="lidar_imu_link"/>
-    <origin xyz="-0.007698 -0.014655 0.00667" rpy="${lidar_imu_roll} ${lidar_imu_pitch} 0"/>
+    <!-- rpy="0 0 0" matches go2_description and DLIO extrinsics convention.
+         The physical IMU tilt within the L1 housing is already compensated by the
+         UniLidar SDK on the real robot; the sim IMU should present the same
+         pre-corrected frame so dlio_params_sim.yaml extrinsics remain valid. -->
+    <origin xyz="-0.007698 -0.014655 0.00667" rpy="0 0 0"/>
   </joint>
   <link name="lidar_imu_link">
@@ -309,12 +313,12 @@
       <imu>
         <angular_velocity>
-          <x><noise type="gaussian"><mean>${lidar_imu_ang_bias_x}</mean><stddev>0.009</stddev></noise></x>
-          <y><noise type="gaussian"><mean>${lidar_imu_ang_bias_y}</mean><stddev>0.009</stddev></noise></y>
-          <z><noise type="gaussian"><mean>${lidar_imu_ang_bias_z}</mean><stddev>0.009</stddev></noise></z>
+          <x><noise type="gaussian"><mean>0.0</mean><stddev>0.009</stddev></noise></x>
+          <y><noise type="gaussian"><mean>0.0</mean><stddev>0.009</stddev></noise></y>
+          <z><noise type="gaussian"><mean>0.0</mean><stddev>0.009</stddev></noise></z>
         </angular_velocity>
         <linear_acceleration>
-          <x><noise type="gaussian"><mean>${lidar_imu_acc_bias_x}</mean><stddev>0.021</stddev></noise></x>
-          <y><noise type="gaussian"><mean>${lidar_imu_acc_bias_y}</mean><stddev>0.021</stddev></noise></y>
-          <z><noise type="gaussian"><mean>${lidar_imu_acc_bias_z}</mean><stddev>0.021</stddev></noise></z>
+          <x><noise type="gaussian"><mean>0.0</mean><stddev>0.021</stddev></noise></x>
+          <y><noise type="gaussian"><mean>0.0</mean><stddev>0.021</stddev></noise></y>
+          <z><noise type="gaussian"><mean>0.0</mean><stddev>0.021</stddev></noise></z>
         </linear_acceleration>
       </imu>

File: src/simulation/sensor_models/urdf/l1_lidar.urdf.xacro (robot description, xacro)
@@ -54,10 +54,4 @@
         </material>
       </visual>
-      <collision>
-        <origin xyz="0 0 0" rpy="0 0 0"/>
-        <geometry>
-          <cylinder radius="0.04" length="0.02"/>
-        </geometry>
-      </collision>
       <inertial>
         <mass value="0.5"/>
