Commit message: - Updated go2_sim.urdf.xacro to improve frame tree structure and added lidar_imu_link for UniLidar IMU integration. - Modified l1_lidar.urdf.xacro to adjust sensor specifications and ensure compatibility with Gazebo Fortress. - Introduced dlio_params_sim.yaml for simulation-specific DLIO parameters to align LiDAR and IMU data. - Created robot_nav package with pointcloud_utils.py for LiDAR point cloud processing and cloud_self_filter.py to filter robot-body returns from PointCloud2 data. - Fixed lidar simulation

File: src/platform/go2_description/urdf/go2.urdf.xacro (robot description, xacro)
@@ -5,11 +5,11 @@
   Frame tree (Nav2 standard contract):
     base_footprint  (published dynamically by the hardware bridge / sim launch)
-      └─ base_link        (robot body center at standing height, roll/pitch-capable)
-           ├─ trunk        (visual/collision body mesh)
-           ├─ imu_link     (co-located with trunk centre)
-           └─ lidar_link   (Unitree L1 LiDAR mount)
+      += base_link        (robot body center at standing height, roll/pitch-capable)
+           += trunk        (visual/collision body mesh)
+           += imu_link     (co-located with trunk centre)
+           += lidar_link   (Unitree L1 LiDAR mount)
   Notes:
     - This URDF is rooted at base_link. base_footprint is intentionally not part of
-      robot_description so bringup can publish base_footprint→base_link dynamically
+      robot_description so bringup can publish base_footprint->base_link dynamically
       from IMU roll/pitch without conflicting with robot_state_publisher.
     - lidar_link pose matches Go2 mounting location used by Nav2/SLAM.
@@ -22,7 +22,7 @@
 -->
 <robot name="go2" xmlns:xacro="http://www.ros.org/wiki/xacro">
-  <!-- ═══════════════════════════════════════════════════════════════════════
+  <!-- =======================================================================
        Physical constants
-  ════════════════════════════════════════════════════════════════════════════ -->
+  ============================================================================ -->
   <xacro:property name="body_length"  value="0.440"/>   <!-- trunk X -->
   <xacro:property name="body_width"   value="0.060"/>   <!-- trunk half-width in Y -->
@@ -44,10 +44,11 @@
   <xacro:property name="lidar_y" value="0.0"/>
   <xacro:property name="lidar_z" value="-0.046825"/>
-  <xacro:property name="lidar_r" value="0.0"/>
-  <xacro:property name="lidar_p" value="0.0"/>
+  <!-- Real Go2 mount: Unitree L1 is upside-down with ~15deg forward pitch. -->
+  <xacro:property name="lidar_r" value="3.14159265358979"/>
+  <xacro:property name="lidar_p" value="-0.26179938779915"/>
   <xacro:property name="lidar_yaw" value="0.0"/>
-  <!-- ═══════════════════════════════════════════════════════════════════════
-       base_link  —  robot body centre
-  ════════════════════════════════════════════════════════════════════════════ -->
+  <!-- =======================================================================
+       base_link  -  robot body centre
+  ============================================================================ -->
   <link name="base_link">
     <visual>
@@ -55,6 +56,6 @@
       <geometry>
         <!--
-          TRUNK ONLY — this box represents the rigid body torso, not the full
-          robot envelope. The full standing footprint (700×310 mm including legs)
+          TRUNK ONLY - this box represents the rigid body torso, not the full
+          robot envelope. The full standing footprint (700x310 mm including legs)
           is represented in Nav2 via the footprint parameter in nav2_params.yaml.
           Replace with mesh when available:
@@ -67,5 +68,5 @@
       </material>
     </visual>
-    <!-- Leg stance envelope — represents the physical standing footprint.
+    <!-- Leg stance envelope - represents the physical standing footprint.
          Positioned at z = -(standing_height - stance_height/2) relative to
          base_link, which is: -(0.28 - 0.115) = -0.165 m -->
@@ -83,6 +84,6 @@
       <geometry>
         <!--
-          TRUNK ONLY — this box represents the rigid body torso, not the full
-          robot envelope. The full standing footprint (700×310 mm including legs)
+          TRUNK ONLY - this box represents the rigid body torso, not the full
+          robot envelope. The full standing footprint (700x310 mm including legs)
           is represented in Nav2 via the footprint parameter in nav2_params.yaml.
           Replace with mesh when available:
@@ -107,7 +108,7 @@
     </inertial>
   </link>
-  <!-- ═══════════════════════════════════════════════════════════════════════
-       imu_link  —  co-located with trunk centre (Go2 internal IMU)
-  ════════════════════════════════════════════════════════════════════════════ -->
+  <!-- =======================================================================
+       imu_link  -  co-located with trunk centre (Go2 internal IMU)
+  ============================================================================ -->
   <joint name="base_link_to_imu" type="fixed">
     <parent link="base_link"/>
@@ -122,8 +123,8 @@
     </inertial>
   </link>
-  <!-- ═══════════════════════════════════════════════════════════════════════
-       lidar_link  —  Unitree L1 LiDAR optical/spinning centre
+  <!-- =======================================================================
+       lidar_link  -  Unitree L1 LiDAR optical/spinning centre
        +X forward, +Y left, +Z up  (standard ROS sensor convention)
-  ════════════════════════════════════════════════════════════════════════════ -->
+  ============================================================================ -->
   <joint name="base_link_to_lidar" type="fixed">
     <parent link="base_link"/>
@@ -147,6 +148,22 @@
     </inertial>
   </link>
-  <!-- FIX(agent5): Removed <gazebo> block that was present in go2_description.
-       All Gazebo material/plugin tags belong exclusively in go2_sim/urdf/go2_sim.urdf.xacro.
-       The use_gazebo xacro:arg is also removed as it is no longer referenced. -->
+  <!-- ====================================================================
+       lidar_imu_link  -  Unitree UniLidar built-in IMU origin
+       Offset within the L1 sensor body, published by robot_state_publisher.
+       lio.launch.py must use publish_lidar_imu_tf:=false on hardware to avoid
+       duplicating this TF.  In simulation this joint is already defined in
+       go2_sim.urdf.xacro; on hardware the URDF is the authoritative source.
+       ==================================================================== -->
+  <joint name="lidar_to_lidar_imu" type="fixed">
+    <parent link="lidar_link"/>
+    <child  link="lidar_imu_link"/>
+    <origin xyz="-0.007698 -0.014655 0.00667" rpy="0 0 0"/>
+  </joint>
+  <link name="lidar_imu_link">
+    <inertial>
+      <mass value="0.001"/>
+      <origin xyz="0 0 0" rpy="0 0 0"/>
+      <inertia ixx="1e-7" ixy="0" ixz="0" iyy="1e-7" iyz="0" izz="1e-7"/>
+    </inertial>
+  </link>
 </robot>

File: src/simulation/go2_sim/urdf/go2_sim.urdf.xacro (robot description, xacro)
@@ -2,16 +2,17 @@
 <!--
   go2_sim.urdf.xacro
-  Unitree Go2 — Gazebo Fortress (Ignition Gazebo 6) + CHAMP simulation model.
+  Unitree Go2 - Gazebo Fortress (Ignition Gazebo 6) + CHAMP simulation model.
   Port contract:
     - Source:  khaledgabr77/unitree_go2_ros2 (Gazebo Harmonic, ROS 2 Jazzy)
     - Target:  go2_sim (Gazebo Fortress / Ignition Gazebo 6, ROS 2 Humble)
   Frame tree:
-    base_link (robot body — matches go2_description and go2_bringup convention)
-      ├── trunk                  (body visual/collision/inertia; floating_base joint)
-      ├── imu_link               (IMU sensor frame)
-      ├── {lf,rf,lh,rh}_hip_link → {lf,rf,lh,rh}_upper_leg_link
-      │                         → {lf,rf,lh,rh}_lower_leg_link
-      │                         → LF_FOOT / RF_FOOT / LH_FOOT / RH_FOOT (CHAMP)
-      └── lidar_link             (Unitree L1 LiDAR; provided by sensor_models macro, prefix="")
+    base_link (robot body - matches go2_description and go2_bringup convention)
+      +== trunk                  (body visual/collision/inertia; floating_base joint)
+      +== imu_link               (IMU sensor frame)
+      +== {lf,rf,lh,rh}_hip_link -> {lf,rf,lh,rh}_upper_leg_link
+      |                         -> {lf,rf,lh,rh}_lower_leg_link
+      |                         -> LF_FOOT / RF_FOOT / LH_FOOT / RH_FOOT (CHAMP)
+      +== lidar_link             (Unitree L1 LiDAR; provided by sensor_models macro, prefix="")
+           += lidar_imu_link    (UniLidar built-in IMU; fixed offset within L1 body)
   CHAMP requires four foot links named exactly: LF_FOOT RF_FOOT LH_FOOT RH_FOOT
   These are generated by the leg macro in leg.xacro.
@@ -21,27 +22,27 @@
     - ignition-gazebo-contact-system   (foot contact sensors)
     - ignition-gazebo-joint-state-publisher-system  (/joint_states)
-    - ignition-gazebo-sensors-system   (gpu_lidar — in world SDF, handles L1)
+    - ignition-gazebo-sensors-system   (gpu_lidar - in world SDF, handles L1)
   Topics published (bridged to ROS via ros_ign_bridge in launch file):
-    /joint_states       — sensor_msgs/JointState
-    /imu/data           — sensor_msgs/Imu
-    /lidar/points     — sensor_msgs/PointCloud2   (gpu_lidar publishes PointCloudPacked on /lidar/points)
-    /cmd_vel            — geometry_msgs/Twist        (ROS → Gazebo)
-    /model/go2/odometry — nav_msgs/Odometry          (Ignition → ROS as /odom/raw → EKF)
-  DO NOT USE gz:: namespaces — Fortress uses ignition:: exclusively.
+    /joint_states       - sensor_msgs/JointState
+    /imu/data           - sensor_msgs/Imu
+    /lidar/points     - sensor_msgs/PointCloud2   (gpu_lidar publishes PointCloudPacked on /lidar/points)
+    /cmd_vel            - geometry_msgs/Twist        (ROS -> Gazebo)
+    /model/go2/odometry - nav_msgs/Odometry          (Ignition -> ROS as /odom/raw -> EKF)
+  DO NOT USE gz:: namespaces - Fortress uses ignition:: exclusively.
 -->
 <robot name="go2"
        xmlns:xacro="http://www.ros.org/wiki/xacro">
-  <!-- ── xacro arguments ── -->
+  <!-- == xacro arguments == -->
   <xacro:arg name="DEBUG"            default="false"/>
   <xacro:arg name="robot_controllers"
              default="$(find go2_sim)/config/ros_control.yaml"/>
-  <!-- ── Include sub-files ── -->
+  <!-- == Include sub-files == -->
   <xacro:include filename="$(find go2_sim)/urdf/const.xacro"/>
   <xacro:include filename="$(find go2_sim)/urdf/materials.xacro"/>
   <xacro:include filename="$(find go2_sim)/urdf/leg.xacro"/>
   <xacro:include filename="$(find sensor_models)/urdf/l1_lidar.urdf.xacro"/>
-  <!-- ════════════════════════════════════════════════════════════════════
+  <!-- ====================================================================
        GAZEBO PLUGINS  (Fortress / ignition:: namespace)
-       ════════════════════════════════════════════════════════════════════ -->
+       ==================================================================== -->
   <!-- ign_ros2_control: loads controller_manager, reads ros_control.yaml -->
   <gazebo>
@@ -60,5 +61,5 @@
   <!-- Ignition odometry publisher: tracks base_link velocity in the world and
        publishes nav_msgs/Odometry on Ignition topic /model/go2/odometry.
-       Bridged to ROS as /odom/raw → EKF (footprint_to_odom_ekf) → /odom + TF. -->
+       Bridged to ROS as /odom/raw -> EKF (footprint_to_odom_ekf) -> /odom + TF. -->
   <gazebo>
     <plugin filename="ignition-gazebo-odometry-publisher-system"
@@ -69,7 +70,7 @@
     </plugin>
   </gazebo>
-  <!-- ════════════════════════════════════════════════════════════════════
+  <!-- ====================================================================
        OPTIONAL DEBUG MODE: pin robot to world for tuning
-       ════════════════════════════════════════════════════════════════════ -->
+       ==================================================================== -->
   <xacro:if value="$(arg DEBUG)">
     <link name="world"/>
@@ -80,7 +81,7 @@
     </joint>
   </xacro:if>
-  <!-- ════════════════════════════════════════════════════════════════════
-       BASE LINK  (virtual root — matches CHAMP expectation)
-       ════════════════════════════════════════════════════════════════════ -->
+  <!-- ====================================================================
+       BASE LINK  (virtual root - matches CHAMP expectation)
+       ==================================================================== -->
   <link name="base_link">
     <visual>
@@ -89,7 +90,7 @@
     </visual>
   </link>
-  <!-- ════════════════════════════════════════════════════════════════════
+  <!-- ====================================================================
        TRUNK  (main body visual / collision / inertia)
-       ════════════════════════════════════════════════════════════════════ -->
+       ==================================================================== -->
   <joint name="floating_base" type="fixed">
     <origin rpy="0 0 0" xyz="0 0 0"/>
@@ -123,7 +124,7 @@
     <kd>1.0</kd>
   </gazebo>
-  <!-- ════════════════════════════════════════════════════════════════════
+  <!-- ====================================================================
        IMU LINK
-       ════════════════════════════════════════════════════════════════════ -->
+       ==================================================================== -->
   <joint name="imu_joint" type="fixed">
     <parent link="trunk"/>
@@ -172,7 +173,7 @@
     </sensor>
   </gazebo>
-  <!-- ════════════════════════════════════════════════════════════════════
-       LEGS  (4× instantiation via leg macro — defines foot links LF/RF/LH/RH_FOOT)
-       ════════════════════════════════════════════════════════════════════ -->
+  <!-- ====================================================================
+       LEGS  (4x instantiation via leg macro - defines foot links LF/RF/LH/RH_FOOT)
+       ==================================================================== -->
   <!--  RF: mirror=-1 (right), mirror_dae=False (right mesh), front_hind=1, front_hind_dae=True  -->
   <xacro:leg name="rf" mirror="-1" mirror_dae="False" front_hind="1"  front_hind_dae="True"/>
@@ -183,5 +184,5 @@
   <!--  LH: mirror=1  (left),  mirror_dae=True  (left mesh),  front_hind=-1, front_hind_dae=False -->
   <xacro:leg name="lh" mirror="1"  mirror_dae="True"  front_hind="-1" front_hind_dae="False"/>
-  <!-- ── Gazebo physics properties for legs ── -->
+  <!-- == Gazebo physics properties for legs == -->
   <!-- LF leg -->
   <gazebo reference="lf_hip_link">       <mu1>0.2</mu1><mu2>0.2</mu2></gazebo>
@@ -204,9 +205,9 @@
   <gazebo reference="rh_lower_leg_link"> <mu1>0.2</mu1><mu2>0.2</mu2><self_collide>1</self_collide></gazebo>
   <gazebo reference="RH_FOOT">           <mu1>0.6</mu1><mu2>0.6</mu2><self_collide>1</self_collide><kp>10000.0</kp><kd>1.0</kd></gazebo>
-  <!-- ════════════════════════════════════════════════════════════════════
+  <!-- ====================================================================
        FOOT CONTACT SENSORS  (Fortress syntax, ignition-gazebo-contact-system)
        One sensor per foot; collision name = <foot_link>_collision (auto-generated
        by Gazebo from the URDF collision element of each foot link).
-       ════════════════════════════════════════════════════════════════════ -->
+       ==================================================================== -->
   <gazebo reference="LF_FOOT">
     <sensor name="LF_FOOT_contact" type="contact">
@@ -241,5 +242,5 @@
     </sensor>
   </gazebo>
-  <!-- ════════════════════════════════════════════════════════════════════
+  <!-- ====================================================================
        L1 LIDAR  (from sensor_models Fortress macro)
        Mount position from source repo reference
@@ -252,9 +253,61 @@
          go2_description       lidar_link frame convention
          nav2_params.yaml      voxel_layer expects /lidar/points in lidar_link
-       ════════════════════════════════════════════════════════════════════ -->
+       ==================================================================== -->
   <xacro:l1_lidar parent="base_link" prefix="">
-    <!-- The Unitree L1 is mounted upside down on Go2, so its upward
-         hemispherical scan in sensor frame points toward the floor. -->
-    <origin xyz="0.28945 0 -0.056825" rpy="3.14159265358979 0 0"/>
+    <!-- Sim-only: right-side-up mount (no Rx(pi) roll) because Fortress
+         gpu_lidar drops most rays when the parent link has a 180-deg roll.
+         Pitch-only rotation replicates the real 15-deg forward tilt.
+         The vertical scan angles in l1_lidar.urdf.xacro are negated to
+         compensate so the point cloud covers the same world region. -->
+    <origin xyz="0.28945 0 -0.046825" rpy="0 -0.26179938779915 0"/>
   </xacro:l1_lidar>
+  <!-- ====================================================================
+       LIDAR IMU LINK  (Unitree UniLidar built-in IMU)
+       Offset within the L1 sensor body; matches go2_description convention.
+       ==================================================================== -->
+  <joint name="lidar_to_lidar_imu" type="fixed">
+    <parent link="lidar_link"/>
+    <child  link="lidar_imu_link"/>
+    <origin xyz="-0.007698 -0.014655 0.00667" rpy="0 0 0"/>
+  </joint>
+  <link name="lidar_imu_link">
+    <inertial>
+      <mass value="0.001"/>
+      <origin xyz="0 0 0" rpy="0 0 0"/>
+      <inertia ixx="1e-7" ixy="0" ixz="0" iyy="1e-7" iyz="0" izz="1e-7"/>
+    </inertial>
+    <visual>
+      <origin rpy="0 0 0" xyz="0 0 0"/>
+      <geometry><box size="0.001 0.001 0.001"/></geometry>
+    </visual>
+    <collision>
+      <origin rpy="0 0 0" xyz="0 0 0"/>
+      <geometry><box size="0.001 0.001 0.001"/></geometry>
+    </collision>
+  </link>
+  <!--
+    UniLidar built-in IMU sensor published on /lidar/imu.
+    Bridged to ROS via ros_ign_bridge in sim_champ.launch.py.
+    System plugin ignition-gazebo-imu-system is loaded in the world SDF.
+  -->
+  <gazebo reference="lidar_imu_link">
+    <sensor name="lidar_imu_sensor" type="imu">
+      <always_on>1</always_on>
+      <update_rate>200</update_rate>
+      <topic>/lidar/imu</topic>
+      <ignition_frame_id>lidar_imu_link</ignition_frame_id>
+      <imu>
+        <angular_velocity>
+          <x><noise type="gaussian"><mean>0</mean><stddev>0.009</stddev></noise></x>
+          <y><noise type="gaussian"><mean>0</mean><stddev>0.009</stddev></noise></y>
+          <z><noise type="gaussian"><mean>0</mean><stddev>0.009</stddev></noise></z>
+        </angular_velocity>
+        <linear_acceleration>
+          <x><noise type="gaussian"><mean>0</mean><stddev>0.021</stddev></noise></x>
+          <y><noise type="gaussian"><mean>0</mean><stddev>0.021</stddev></noise></y>
+          <z><noise type="gaussian"><mean>0</mean><stddev>0.021</stddev></noise></z>
+        </linear_acceleration>
+      </imu>
+    </sensor>
+  </gazebo>
 </robot>
