Commit message: refactor(go2): consolidate leg URDF in go2_description; publish /joint_states from lowstate
URDF consolidation
- Move Go2 mesh + shared xacros (const.xacro, leg.xacro, materials.xacro)
  from go2_sim to go2_description so the hardware URDF has articulated
  legs for RViz and both sim and real reference the same source of truth.
- go2.urdf.xacro: instantiate leg macros (with_ros2_control off on
  hardware) so robot_state_publisher animates leg links from
  /joint_states. Keep base_link collision boxes for Nav2 footprint use.
- go2_sim.urdf.xacro: switch includes and mesh URIs to point at
  go2_description; go2_sim package.xml gains go2_description exec_depend.
- Drop unused base.dae.bak files.

Hardware /joint_states
- go2_hw_bridge decimates /lowstate motor_state[0..11] to
  sensor_msgs/JointState at 50 Hz (parameter joint_states_rate). Motor
  indices mapped to CHAMP-style joint names (FR=0..2, FL=3..5, RR=6..8,
  RL=9..11 with 0=hip, 1=thigh, 2=calf).
- docs/topic_map.md: updated /joint_states row to reflect the HW path.

Co-Authored-By: Claude Opus 4.7 (1M context) <noreply@anthropic.com>

File: src/platform/go2_description/urdf/go2.urdf.xacro (robot description, xacro)
@@ -2,24 +2,34 @@
 <!--
   go2.urdf.xacro
-  Minimal Go2 robot description for Nav2 navigation.
+  Hardware Go2 robot description for Nav2 navigation and RViz visualization.
   Frame tree (Nav2 standard contract):
     base_footprint  (published dynamically by the hardware bridge / sim launch)
-      += base_link        (robot body center at standing height, roll/pitch-capable)
-           += trunk        (visual/collision body mesh)
-           += imu_link     (co-located with trunk centre)
-           += lidar_link   (Unitree L1 LiDAR mount)
+      += base_link             (robot body center at standing height, roll/pitch-capable)
+           += trunk             (Go2 body mesh; fixed offset, identity)
+           |    += {lf,rf,lh,rh}_hip_link -> {..}_upper_leg_link -> {..}_lower_leg_link -> {LF,RF,LH,RH}_FOOT
+           += imu_link          (co-located with trunk centre)
+           += lidar_link        (Unitree L1 LiDAR mount, real driver orientation)
   Notes:
     - This URDF is rooted at base_link. base_footprint is intentionally not part of
       robot_description so bringup can publish base_footprint->base_link dynamically
       from IMU roll/pitch without conflicting with robot_state_publisher.
-    - lidar_link pose matches Go2 mounting location used by Nav2/SLAM.
-    - Leg links are omitted (not needed for Nav2). Add them when joint-state
-      visualization or IK is required.
-  NOTE: Gazebo simulation plugins are implemented in go2_sim/urdf/go2_sim.urdf.xacro.
-        This hardware-focused URDF intentionally keeps simulation plugins out.
+    - lidar_link pose matches the Go2 mounting location used by Nav2/SLAM (real
+      driver orientation; see go2_sim/urdf/go2_sim.urdf.xacro for the Fortress
+      workaround used in simulation).
+    - Leg links + joints are present so RViz mirrors the real robot pose when
+      go2_hw_bridge publishes /joint_states from /lowstate.motor_state[].q. The
+      ros2_control block from leg.xacro is gated off here (hardware does not use
+      ign_ros2_control).
+    - base_link keeps two collision boxes (trunk + safety envelope) so Nav2
+      consumers that read URDF collision geometry get the standing footprint
+      independent of leg articulation.
   TODO(agibot): Create agibot_d1_description/urdf/d1.urdf.xacro with the same
                 frame names (base_footprint, base_link, lidar_link, imu_link).
 -->
 <robot name="go2" xmlns:xacro="http://www.ros.org/wiki/xacro">
+  <!-- Shared geometry: leg/joint constants, mesh materials, parametric leg macro. -->
+  <xacro:include filename="$(find go2_description)/urdf/const.xacro"/>
+  <xacro:include filename="$(find go2_description)/urdf/materials.xacro"/>
+  <xacro:include filename="$(find go2_description)/urdf/leg.xacro"/>
   <!-- =======================================================================
        Physical constants
@@ -49,45 +59,15 @@
   <xacro:property name="lidar_yaw" value="0.0"/>
   <!-- =======================================================================
-       base_link  -  robot body centre
+       base_link  -  virtual root + Nav2 collision geometry
+       Visuals live on `trunk` (Go2 body mesh) and the leg links instantiated
+       below. The collision boxes here express the full standing footprint for
+       Nav2 consumers that read URDF collision geometry.
   ============================================================================ -->
   <link name="base_link">
-    <visual>
-      <origin xyz="0 0 0" rpy="0 0 0"/>
-      <geometry>
-        <!--
-          TRUNK ONLY - this box represents the rigid body torso, not the full
-          robot envelope. The full standing footprint (700x310 mm including legs)
-          is represented in Nav2 via the footprint parameter in nav2_params.yaml.
-          Replace with mesh when available:
-            <mesh filename="file://$(find go2_description)/meshes/trunk.dae"/>
-        -->
-        <box size="${body_length} ${body_width*2} ${body_height}"/>
-      </geometry>
-      <material name="dark_grey">
-        <color rgba="0.2 0.2 0.2 1.0"/>
-      </material>
-    </visual>
-    <!-- Leg stance envelope - represents the physical standing footprint.
-         Positioned at z = -(standing_height - stance_height/2) relative to
-         base_link, which is: -(0.28 - 0.115) = -0.165 m -->
-    <visual name="stance_visual">
-      <origin xyz="0 0 ${-(standing_height - stance_height/2)}" rpy="0 0 0"/>
-      <geometry>
-        <box size="${stance_length} ${stance_width} ${stance_height}"/>
-      </geometry>
-      <material name="stance_grey">
-        <color rgba="0.5 0.5 0.5 0.4"/>
-      </material>
-    </visual>
     <collision>
       <origin xyz="0 0 0" rpy="0 0 0"/>
       <geometry>
-        <!--
-          TRUNK ONLY - this box represents the rigid body torso, not the full
-          robot envelope. The full standing footprint (700x310 mm including legs)
-          is represented in Nav2 via the footprint parameter in nav2_params.yaml.
-          Replace with mesh when available:
-            <mesh filename="file://$(find go2_description)/meshes/trunk.dae"/>
-        -->
+        <!-- Rigid body torso footprint (full standing envelope is via the
+             safety collision below and nav2 footprint parameters). -->
         <box size="${body_length} ${body_width*2} ${body_height}"/>
       </geometry>
@@ -100,12 +80,39 @@
       </geometry>
     </collision>
+  </link>
+  <!-- =======================================================================
+       trunk  -  Go2 body mesh, fixed offset from base_link
+       Matches the sim URDF (go2_sim.urdf.xacro) so RViz appearance and the leg
+       attachment frame are identical between sim and real.
+  ============================================================================ -->
+  <joint name="floating_base" type="fixed">
+    <parent link="base_link"/>
+    <child  link="trunk"/>
+    <origin xyz="0 0 0" rpy="0 0 0"/>
+  </joint>
+  <link name="trunk">
+    <visual>
+      <origin xyz="0 0 0" rpy="0 0 0"/>
+      <geometry>
+        <mesh filename="package://go2_description/meshes/dae/base.dae" scale="1 1 1"/>
+      </geometry>
+    </visual>
     <inertial>
-      <origin xyz="0.021112 0.0 -0.005366" rpy="0 0 0"/>
-      <mass value="${body_mass}"/>
-      <inertia ixx="0.02448"  ixy="0.00012166" ixz="0.0014849"
-               iyy="0.098077" iyz="-0.0000312"
-               izz="0.107"/>
+      <origin xyz="${trunk_com_x} ${trunk_com_y} ${trunk_com_z}" rpy="0 0 0"/>
+      <mass value="${trunk_mass}"/>
+      <inertia ixx="${trunk_ixx}" ixy="${trunk_ixy}" ixz="${trunk_ixz}"
+               iyy="${trunk_iyy}" iyz="${trunk_iyz}"
+               izz="${trunk_izz}"/>
     </inertial>
   </link>
+  <!-- =======================================================================
+       Articulated legs - joint_states fed by go2_hw_bridge from /lowstate.
+       Same macro and mirroring scheme as the sim URDF; ros2_control block is
+       gated off (hardware does not use ign_ros2_control).
+  ============================================================================ -->
+  <xacro:leg name="rf" mirror="-1" mirror_dae="False" front_hind="1"  front_hind_dae="True"  parent="trunk" with_ros2_control="False"/>
+  <xacro:leg name="lf" mirror="1"  mirror_dae="True"  front_hind="1"  front_hind_dae="True"  parent="trunk" with_ros2_control="False"/>
+  <xacro:leg name="rh" mirror="-1" mirror_dae="False" front_hind="-1" front_hind_dae="False" parent="trunk" with_ros2_control="False"/>
+  <xacro:leg name="lh" mirror="1"  mirror_dae="True"  front_hind="-1" front_hind_dae="False" parent="trunk" with_ros2_control="False"/>
   <!-- =======================================================================
        imu_link  -  co-located with trunk centre (Go2 internal IMU)

File: src/platform/go2_description/urdf/leg.xacro (robot description, xacro)
@@ -2,21 +2,25 @@
 <!--
   leg.xacro
-  Parametric leg macro for the Unitree Go2 (Gazebo Fortress / ign_ros2_control).
+  Parametric leg macro for the Unitree Go2.
   Source: khaledgabr77/unitree_go2_ros2 / unitree_go2_description/urdf/leg.xacro
   Changes vs. source:
-    1. Foot link names renamed: {name}_foot_link → uppercase CHAMP convention
-         lf → LF_FOOT,  rf → RF_FOOT,  lh → LH_FOOT,  rh → RH_FOOT
+    1. Foot link names renamed: {name}_foot_link -> uppercase CHAMP convention
+         lf -> LF_FOOT,  rf -> RF_FOOT,  lh -> LH_FOOT,  rh -> RH_FOOT
        Joint child references updated accordingly.
-    2. ros2_control hardware plugin changed:
-         Fortress control interface plugin → ign_ros2_control/IgnitionSystem
-    3. Mesh paths changed:
-         package://unitree_go2_description/meshes/ → package://go2_sim/meshes/dae/
-    4. Typo in source fixed: line had `type="fixed">0` — the stray `0` removed.
-  Macro parameters (unchanged from source):
-    name         — leg prefix: lf | rf | lh | rh
-    mirror       — Y-axis sign:  1 (left) | -1 (right)
-    mirror_dae   — True (left, use original mesh) | False (right, use mirrored mesh)
-    front_hind   — X-axis sign:  1 (front) | -1 (hind)
-    front_hind_dae — True (front) | False (hind)
+    2. Mesh paths now resolve against go2_description (shared between sim and real).
+    3. ros2_control block is sim-only and gated by the `with_ros2_control` macro
+       parameter so hardware bringup gets pure URDF without the Fortress plugin.
+    4. Hip joint parent link is parameterized (`parent` argument) so both the sim
+       URDF (parent="trunk") and the hardware URDF (parent="trunk") can reuse this
+       macro without duplicating geometry.
+    5. Typo in source fixed: line had `type="fixed">0` - the stray `0` removed.
+  Macro parameters:
+    name              - leg prefix: lf | rf | lh | rh
+    mirror            - Y-axis sign:  1 (left) | -1 (right)
+    mirror_dae        - True (left, use original mesh) | False (right, use mirrored mesh)
+    front_hind        - X-axis sign:  1 (front) | -1 (hind)
+    front_hind_dae    - True (front) | False (hind)
+    parent            - parent link for the hip joint (default: "trunk")
+    with_ros2_control - emit `<ros2_control>` block for Gazebo (default: "false")
 -->
 <robot xmlns:xacro="http://www.ros.org/wiki/xacro">
@@ -29,5 +33,5 @@
       The xacro property below derives the CHAMP name from the leg prefix.
     -->
-    <xacro:macro name="leg" params="name mirror mirror_dae front_hind front_hind_dae">
+    <xacro:macro name="leg" params="name mirror mirror_dae front_hind front_hind_dae parent:=^|'trunk' with_ros2_control:=^|False">
         <!-- Derive CHAMP-convention foot link name from leg prefix -->
         <xacro:if value="${name == 'lf'}">
@@ -57,5 +61,5 @@
                 <origin rpy="0 0 0" xyz="${-leg_offset_x} ${leg_offset_y} 0"/>
             </xacro:if>
-            <parent link="trunk"/>
+            <parent link="${parent}"/>
             <child link="${name}_hip_link"/>
             <axis xyz="1 0 0"/>
@@ -86,5 +90,5 @@
                 </xacro:if>
                 <geometry>
-                    <mesh filename="package://go2_sim/meshes/dae/hip.dae" scale="1 1 1"/>
+                    <mesh filename="package://go2_description/meshes/dae/hip.dae" scale="1 1 1"/>
                 </geometry>
             </visual>
@@ -124,8 +128,8 @@
                 <geometry>
                     <xacro:if value="${mirror_dae == True}">
-                        <mesh filename="package://go2_sim/meshes/dae/thigh.dae" scale="1 1 1"/>
+                        <mesh filename="package://go2_description/meshes/dae/thigh.dae" scale="1 1 1"/>
                     </xacro:if>
                     <xacro:if value="${mirror_dae == False}">
-                        <mesh filename="package://go2_sim/meshes/dae/thigh_mirror.dae" scale="1 1 1"/>
+                        <mesh filename="package://go2_description/meshes/dae/thigh_mirror.dae" scale="1 1 1"/>
                     </xacro:if>
                 </geometry>
@@ -165,5 +169,5 @@
                 <origin rpy="0 0 0" xyz="0 0 0"/>
                 <geometry>
-                    <mesh filename="package://go2_sim/meshes/dae/calf.dae" scale="1 1 1"/>
+                    <mesh filename="package://go2_description/meshes/dae/calf.dae" scale="1 1 1"/>
                 </geometry>
             </visual>
@@ -217,25 +221,27 @@
             </inertial>
         </link>
-        <!-- ── ros2_control interface (Fortress: ign_ros2_control/IgnitionSystem) ── -->
-        <ros2_control name="${name}" type="system">
-            <hardware>
-                <plugin>ign_ros2_control/IgnitionSystem</plugin>
-            </hardware>
-            <joint name="${name}_hip_joint">
-                <command_interface name="effort"/>
-                <state_interface name="position"/>
-                <state_interface name="velocity"/>
-            </joint>
-            <joint name="${name}_upper_leg_joint">
-                <command_interface name="effort"/>
-                <state_interface name="position"/>
-                <state_interface name="velocity"/>
-            </joint>
-            <joint name="${name}_lower_leg_joint">
-                <command_interface name="effort"/>
-                <state_interface name="position"/>
-                <state_interface name="velocity"/>
-            </joint>
-        </ros2_control>
+        <!-- Gazebo-only ros2_control block (gated; hardware URDF omits it). -->
+        <xacro:if value="${with_ros2_control == True}">
+            <ros2_control name="${name}" type="system">
+                <hardware>
+                    <plugin>ign_ros2_control/IgnitionSystem</plugin>
+                </hardware>
+                <joint name="${name}_hip_joint">
+                    <command_interface name="effort"/>
+                    <state_interface name="position"/>
+                    <state_interface name="velocity"/>
+                </joint>
+                <joint name="${name}_upper_leg_joint">
+                    <command_interface name="effort"/>
+                    <state_interface name="position"/>
+                    <state_interface name="velocity"/>
+                </joint>
+                <joint name="${name}_lower_leg_joint">
+                    <command_interface name="effort"/>
+                    <state_interface name="position"/>
+                    <state_interface name="velocity"/>
+                </joint>
+            </ros2_control>
+        </xacro:if>
     </xacro:macro>
 </robot>

File: src/simulation/go2_sim/urdf/go2_sim.urdf.xacro (robot description, xacro)
@@ -47,8 +47,8 @@
   <xacro:property name="lidar_imu_roll" value="0.194961"/>
   <xacro:property name="lidar_imu_pitch" value="0.144193"/>
-  <!-- == Include sub-files == -->
-  <xacro:include filename="$(find go2_sim)/urdf/const.xacro"/>
-  <xacro:include filename="$(find go2_sim)/urdf/materials.xacro"/>
-  <xacro:include filename="$(find go2_sim)/urdf/leg.xacro"/>
+  <!-- == Include sub-files (shared sources of truth live in go2_description) == -->
+  <xacro:include filename="$(find go2_description)/urdf/const.xacro"/>
+  <xacro:include filename="$(find go2_description)/urdf/materials.xacro"/>
+  <xacro:include filename="$(find go2_description)/urdf/leg.xacro"/>
   <xacro:include filename="$(find sensor_models)/urdf/l1_lidar.urdf.xacro"/>
   <!-- ====================================================================
@@ -112,5 +112,5 @@
       <origin rpy="0 0 0" xyz="0 0 0"/>
       <geometry>
-        <mesh filename="package://go2_sim/meshes/dae/base.dae" scale="1 1 1"/>
+        <mesh filename="package://go2_description/meshes/dae/base.dae" scale="1 1 1"/>
       </geometry>
     </visual>
@@ -187,11 +187,11 @@
        ==================================================================== -->
   <!--  RF: mirror=-1 (right), mirror_dae=False (right mesh), front_hind=1, front_hind_dae=True  -->
-  <xacro:leg name="rf" mirror="-1" mirror_dae="False" front_hind="1"  front_hind_dae="True"/>
+  <xacro:leg name="rf" mirror="-1" mirror_dae="False" front_hind="1"  front_hind_dae="True"  parent="trunk" with_ros2_control="True"/>
   <!--  LF: mirror=1  (left),  mirror_dae=True  (left mesh),  front_hind=1, front_hind_dae=True  -->
-  <xacro:leg name="lf" mirror="1"  mirror_dae="True"  front_hind="1"  front_hind_dae="True"/>
+  <xacro:leg name="lf" mirror="1"  mirror_dae="True"  front_hind="1"  front_hind_dae="True"  parent="trunk" with_ros2_control="True"/>
   <!--  RH: mirror=-1 (right), mirror_dae=False (right mesh), front_hind=-1, front_hind_dae=False -->
-  <xacro:leg name="rh" mirror="-1" mirror_dae="False" front_hind="-1" front_hind_dae="False"/>
+  <xacro:leg name="rh" mirror="-1" mirror_dae="False" front_hind="-1" front_hind_dae="False" parent="trunk" with_ros2_control="True"/>
   <!--  LH: mirror=1  (left),  mirror_dae=True  (left mesh),  front_hind=-1, front_hind_dae=False -->
-  <xacro:leg name="lh" mirror="1"  mirror_dae="True"  front_hind="-1" front_hind_dae="False"/>
+  <xacro:leg name="lh" mirror="1"  mirror_dae="True"  front_hind="-1" front_hind_dae="False" parent="trunk" with_ros2_control="True"/>
   <!-- == Gazebo physics properties for legs == -->
   <!-- LF leg -->
