Commit message: feat(a2w_description): use the official Unitree A2-W URDF
Vendor Unitree's A2W_Description (a2_wheel.urdf + meshes, BSD) as
a2w_upstream.urdf and generate a2w_body.urdf.xacro from it: official calf
(1.751 kg with wheel motor), wheel links (0.982 kg, tyre r 0.0948 m, 0.0494 m
outboard) and <LEG>_wheel_joint (24.5 Nm). Wheel mesh collisions become fitted
cylinders and the debug sphere visuals are dropped. Sensor frames still come from
the legged A2 URDF, which the official A2-W file lacks.

File: src/platform/a2w_description/urdf/a2w.urdf.xacro (robot description, xacro)
@@ -1,12 +1,12 @@
 <?xml version="1.0"?>
 <!--
-  a2w.urdf.xacro - Unitree A2-W (Pro): A2 body + 4 wheels + front/rear Hesai JT128.
-  The A2-W has no public model. Body, legs and the two LiDAR mounts come from the
-  official A2 URDF (a2w_body.urdf.xacro, generated). Wheel size and position are
-  estimates (190 mm tyre at the calf tip, Go2-W / B2-W layout); correct
-  wheel_radius / wheel_offset_y once measured.
+  a2w.urdf.xacro - Unitree A2-W (Pro): official A2-W body/legs/wheels + front/rear LiDAR.
+  Body, legs and wheels come from the official Unitree A2-W URDF (a2w_body.urdf.xacro,
+  generated from a2w_upstream.urdf; wheel joints <LEG>_wheel_joint). That file has no
+  sensor frames, so the LiDAR and camera mounts below are taken from the legged A2
+  URDF (a2_upstream.urdf, unitree_ros), which shares the A2-W body shell.
   fixed_legs:=false (real): leg joints are revolute and follow /joint_states.
-  fixed_legs:=true  (sim):  leg joints are fixed in the standing pose below, so the
-                            URDF->SDF conversion lumps the robot into one base_link.
+  fixed_legs:=true  (sim):  leg and wheel joints are fixed in the standing pose below,
+                            so the URDF->SDF conversion lumps the robot into one base_link.
   Frames added for the autonomy stack (docs/topic_map.md, A2-W section):
     imu_link          body IMU at the base origin
@@ -21,13 +21,10 @@
   <xacro:property name="fixed_legs" value="$(arg fixed_legs)"/>
   <xacro:property name="leg_joint_type" value="${'fixed' if fixed_legs else 'revolute'}"/>
-  <!-- Standing pose (rad). Base height = calf-tip depth + wheel_radius
-       = 0.275*(cos(0.8) + cos(0.7)) + 0.095 ~= 0.497 m. -->
+  <xacro:property name="wheel_joint_type" value="${'fixed' if fixed_legs else 'continuous'}"/>
+  <!-- Standing pose (rad). Base height = wheel-axle depth + tyre radius
+       = 0.275*(cos(0.8) + cos(0.7)) + 0.0948 ~= 0.497 m. -->
   <xacro:property name="stand_hip"   value="0.0"/>
   <xacro:property name="stand_thigh" value="0.8"/>
   <xacro:property name="stand_calf"  value="-1.5"/>
-  <xacro:property name="wheel_radius"   value="0.095"/>
-  <xacro:property name="wheel_width"    value="0.051"/>
-  <xacro:property name="wheel_offset_y" value="0.06"/>
-  <xacro:property name="wheel_mass"     value="1.0"/>
   <xacro:macro name="leg_angles" params="leg">
     <xacro:property name="${leg}_q_hip"   value="${stand_hip if fixed_legs else 0.0}" scope="parent"/>
@@ -40,34 +37,4 @@
   <xacro:leg_angles leg="RR"/>
   <xacro:include filename="$(find a2w_description)/urdf/a2w_body.urdf.xacro"/>
-  <!-- Wheels: continuous about +y at the calf tip, offset outward like the Go2-W.
-       In sim the wheel joints are fixed (the base slides; wheels are visual). -->
-  <xacro:macro name="wheel" params="leg side">
-    <link name="${leg}_foot">
-      <inertial>
-        <mass value="${wheel_mass}"/>
-        <origin xyz="0 0 0" rpy="0 0 0"/>
-        <inertia ixx="0.0025" ixy="0" ixz="0" iyy="0.0045" iyz="0" izz="0.0025"/>
-      </inertial>
-      <visual>
-        <origin xyz="0 0 0" rpy="${pi/2} 0 0"/>
-        <geometry><cylinder radius="${wheel_radius}" length="${wheel_width}"/></geometry>
-        <material name="a2w_tyre"><color rgba="0.12 0.12 0.12 1"/></material>
-      </visual>
-      <collision>
-        <origin xyz="0 0 0" rpy="${pi/2} 0 0"/>
-        <geometry><cylinder radius="${wheel_radius}" length="${wheel_width}"/></geometry>
-      </collision>
-    </link>
-    <joint name="${leg}_foot_joint" type="${'fixed' if fixed_legs else 'continuous'}">
-      <parent link="${leg}_calf"/>
-      <child link="${leg}_foot"/>
-      <origin xyz="0 ${side * wheel_offset_y} -0.275" rpy="0 0 0"/>
-      <axis xyz="0 1 0"/>
-    </joint>
-  </xacro:macro>
-  <xacro:wheel leg="FL" side="1"/>
-  <xacro:wheel leg="FR" side="-1"/>
-  <xacro:wheel leg="RL" side="1"/>
-  <xacro:wheel leg="RR" side="-1"/>
   <!-- Sensor frames. Tiny inertials keep them through URDF->SDF fixed-joint lumping. -->
   <xacro:macro name="sensor_frame" params="name parent xyz rpy">

File: src/platform/a2w_description/urdf/a2w_body.urdf.xacro (robot description, xacro)
@@ -1,7 +1,7 @@
 <?xml version="1.0"?>
-<!-- GENERATED by scripts/generate_a2w_xacro.py from a2_upstream.urdf
-     (unitree_ros, BSD-3-Clause). Do not edit by hand.
-     Requires properties: leg_joint_type and <LEG>_q_<hip|thigh|calf>
-     (set by a2w.urdf.xacro). -->
+<!-- GENERATED by scripts/generate_a2w_xacro.py from a2w_upstream.urdf
+     (official Unitree A2-W description, BSD). Do not edit by hand.
+     Requires properties: leg_joint_type, wheel_joint_type and
+     <LEG>_q_<hip|thigh|calf> (set by a2w.urdf.xacro). -->
 <robot xmlns:xacro="http://www.ros.org/wiki/xacro" name="a2w_body">
   <link name="base_link">
@@ -9,5 +9,5 @@
       <origin xyz="6.982591E-03 -0.712858E-03 12.889523E-03" rpy="0 0 0" />
       <mass value="19.651" />
-      <inertia ixx="141775328.248061E-09" ixy="400505.020171E-09" ixz="-6996487.718114E-09" iyy="407724601.564754E-09" iyz="-361858.857563E-09" izz="472247985.516800E-09" />
+      <inertia ixx="141775.328248061E-06" ixy="400.505020171E-06" ixz="-6996.487718114E-06" iyy="407724.601564754E-06" iyz="-361.858857563E-06" izz="472247.985516800E-06" />
     </inertial>
     <visual>
@@ -21,34 +21,70 @@
     </visual>
     <collision>
-      <origin xyz="0 0 0.007" rpy="0 0 0" />
-      <geometry>
-        <box size="0.24 0.28 0.17" />
-      </geometry>
-    </collision>
-    <collision>
-      <origin xyz="0.25 0 0.119" rpy="0.0 0 0.0" />
-      <geometry>
-        <box size="0.08 0.05 0.02" />
-      </geometry>
-    </collision>
-    <collision>
-      <origin xyz="-0.22 0 0.119" rpy="-0.0 -0.03 0.0" />
-      <geometry>
-        <box size="0.05 0.03 0.016" />
-      </geometry>
-    </collision>
+      <origin xyz="0 0 0.01" rpy="0 0 0" />
+      <geometry>
+        <box size="0.24 0.28 0.16" />
+      </geometry>
+    </collision>
+  </link>
+  <link name="front_bumper">
+    <inertial>
+      <origin xyz="0 0 0" rpy="0 0 0" />
+      <mass value="0.01" />
+      <inertia ixx="0.001" ixy="0" ixz="0" iyy="0.001" iyz="0" izz="0.001" />
+    </inertial>
     <collision>
       <origin xyz="0.365 0 0.1" rpy="0 -0.7 0" />
       <geometry>
-        <box size="0.06 0.1 0.01" />
-      </geometry>
-    </collision>
-    <collision>
-      <origin xyz="-0.31 0 0.112" rpy="0 0.7 0" />
-      <geometry>
-        <box size="0.045 0.1 0.01" />
-      </geometry>
-    </collision>
-  </link>
+        <box size="0.05 0.1 0.01" />
+      </geometry>
+    </collision>
+    <collision>
+      <origin xyz="0.345 0 0.08" rpy="0 -0.0 0" />
+      <geometry>
+        <sphere radius="0.04" />
+      </geometry>
+    </collision>
+    <collision>
+      <origin xyz="0.25 0 0.09" rpy="0 -0.0 0" />
+      <geometry>
+        <sphere radius="0.04" />
+      </geometry>
+    </collision>
+  </link>
+  <joint name="front_bumper_joint" type="fixed" dont_collapse="true">
+    <origin xyz="0.0 0 0" rpy="0 0 0" />
+    <parent link="base_link" />
+    <child link="front_bumper" />
+  </joint>
+  <link name="rear_bumper">
+    <inertial>
+      <origin xyz="0 0 0" rpy="0 0 0" />
+      <mass value="0.01" />
+      <inertia ixx="0.001" ixy="0" ixz="0" iyy="0.001" iyz="0" izz="0.001" />
+    </inertial>
+    <collision>
+      <origin xyz="-0.302 0 0.112" rpy="0 0.7 0" />
+      <geometry>
+        <box size="0.05 0.1 0.01" />
+      </geometry>
+    </collision>
+    <collision>
+      <origin xyz="-0.285 0 0.08" rpy="0 -0.0 0" />
+      <geometry>
+        <sphere radius="0.04" />
+      </geometry>
+    </collision>
+    <collision>
+      <origin xyz="-0.19 0 0.09" rpy="0 -0.0 0" />
+      <geometry>
+        <sphere radius="0.04" />
+      </geometry>
+    </collision>
+  </link>
+  <joint name="rear_bumper_joint" type="fixed" dont_collapse="true">
+    <origin xyz="0.0 0 0" rpy="0 0 0" />
+    <parent link="base_link" />
+    <child link="rear_bumper" />
+  </joint>
   <link name="FL_hip">
     <inertial>
@@ -66,4 +102,16 @@
       </material>
     </visual>
+    <collision>
+      <origin xyz="0.0 0.085 0" rpy="1.571 0 0" />
+      <geometry>
+        <cylinder radius="0.046" length="0.12" />
+      </geometry>
+    </collision>
+    <collision>
+      <origin xyz="0.0 -0.01 0" rpy="1.571 0 0" />
+      <geometry>
+        <cylinder radius="0.045" length="0.06" />
+      </geometry>
+    </collision>
   </link>
   <joint name="FL_hip_joint" type="${leg_joint_type}">
@@ -90,19 +138,13 @@
     </visual>
     <collision>
-      <origin xyz="0.0 -0.04 0" rpy="1.571 0 0" />
-      <geometry>
-        <cylinder radius="0.048" length="0.12" />
-      </geometry>
-    </collision>
-    <collision>
-      <origin xyz="-0.025 0.00 -0.09" rpy="0 0.01 0" />
-      <geometry>
-        <box size="0.055 0.036 0.17" />
-      </geometry>
-    </collision>
-    <collision>
-      <origin xyz="-0.022 0.00 -0.27" rpy="0 -0.75 0" />
-      <geometry>
-        <box size="0.017 0.05 0.05" />
+      <origin xyz="-0.025 -0.003 -0.12" rpy="0 0.0 0" />
+      <geometry>
+        <box size="0.046 0.046 0.14" />
+      </geometry>
+    </collision>
+    <collision>
+      <origin xyz="-0.022 0.00 -0.275" rpy="0 -0.75 0" />
+      <geometry>
+        <box size="0.017 0.05 0.06" />
       </geometry>
     </collision>
@@ -117,7 +159,7 @@
   <link name="FL_calf">
     <inertial>
-      <origin xyz="12.515E-03 -0.024E-03 -117.649E-03" rpy="0 0 0" />
-      <mass value="0.361" />
-      <inertia ixx="3869.035E-06" ixy="-0.093E-06" ixz="298.636E-06" iyy="3945.295E-06" iyz="0.826E-06" izz="150.991E-06" />
+      <origin xyz="4.018E-03 17.411E-03 -232.283E-03" rpy="0 0 0" />
+      <mass value="1.751" />
+      <inertia ixx="14397.534E-06" ixy="124.726E-06" ixz="-550.242E-06" iyy="14603.730E-06" iyz="1307.539E-06" izz="1498.341E-06" />
     </inertial>
     <visual>
@@ -127,11 +169,17 @@
       </geometry>
       <material name="">
-        <color rgba="0.898039215686275 0.917647058823529 0.929411764705882 1" />
-      </material>
-    </visual>
-    <collision>
-      <origin xyz="0.018 -0.00 -0.08" rpy="0 -0.24 0" />
-      <geometry>
-        <box size="0.024 0.03 0.1" />
+        <color rgba="0.792156862745098 0.819607843137255 0.933333333333333 1" />
+      </material>
+    </visual>
+    <collision>
+      <origin xyz="0.0 0.0 -0.275" rpy="1.571 0 0" />
+      <geometry>
+        <cylinder radius="0.05" length="0.03" />
+      </geometry>
+    </collision>
+    <collision>
+      <origin xyz="0.02 -0.00 -0.08" rpy="0 -0.24 0" />
+      <geometry>
+        <box size="0.022 0.03 0.1" />
       </geometry>
     </collision>
@@ -143,13 +191,7 @@
     </collision>
     <collision>
-      <origin xyz="0.029 -0.00 -0.236" rpy="0 0.2 0" />
-      <geometry>
-        <box size="0.02 0.036 0.06" />
-      </geometry>
-    </collision>
-    <collision>
-      <origin xyz="0.008 -0.00 -0.23" rpy="0 0.68 0" />
-      <geometry>
-        <box size="0.01 0.036 0.06" />
+      <origin xyz="0.027 -0.00 -0.23" rpy="0 0.2 0" />
+      <geometry>
+        <box size="0.028 0.04 0.04" />
       </geometry>
     </collision>
@@ -162,4 +204,33 @@
     <limit lower="-2.77" upper="-0.54" effort="180.0" velocity="14.6667" />
   </joint>
+  <link name="FL_wheel">
+    <inertial>
+      <origin xyz="0E-03 51.080E-03 0E-03" rpy="0 0 0" />
+      <mass value="0.982" />
+      <inertia ixx="2435.762E-06" ixy="0E-06" ixz="0E-06" iyy="4581.589E-06" iyz="0E-06" izz="2435.762E-06" />
+    </inertial>
+    <visual>
+      <origin xyz="0 0 0" rpy="0 0 0" />
+      <geometry>
+        <mesh filename="package://a2w_description/meshes/left_front_Link4.STL" />
+      </geometry>
+      <material name="">
+        <color rgba="0.792156862745098 0.819607843137255 0.933333333333333 1" />
+      </material>
+    </visual>
+    <collision>
+      <origin xyz="0 0.0494 0" rpy="1.5708 0 0" />
+      <geometry>
+        <cylinder radius="0.0948" length="0.050" />
+      </geometry>
+    </collision>
+  </link>
+  <joint name="FL_wheel_joint" type="${wheel_joint_type}">
+    <origin xyz="0 0 -0.275" rpy="0 0 0" />
+    <parent link="FL_calf" />
+    <child link="FL_wheel" />
+    <axis xyz="0 1 0" />
+    <limit effort="24.5" velocity="114.4" />
+  </joint>
   <link name="RL_hip">
     <inertial>
@@ -177,4 +248,16 @@
       </material>
     </visual>
+    <collision>
+      <origin xyz="0.0 0.085 0" rpy="1.571 0 0" />
+      <geometry>
+        <cylinder radius="0.046" length="0.12" />
+      </geometry>
+    </collision>
+    <collision>
+      <origin xyz="0.0 -0.01 0" rpy="1.571 0 0" />
+      <geometry>
+        <cylinder radius="0.045" length="0.06" />
+      </geometry>
+    </collision>
   </link>
   <joint name="RL_hip_joint" type="${leg_joint_type}">
@@ -201,19 +284,13 @@
     </visual>
     <collision>
-      <origin xyz="0.0 -0.04 0" rpy="1.571 0 0" />
-      <geometry>
-        <cylinder radius="0.048" length="0.12" />
-      </geometry>
-    </collision>
-    <collision>
-      <origin xyz="-0.025 0.00 -0.09" rpy="0 0.01 0" />
-      <geometry>
-        <box size="0.055 0.036 0.17" />
-      </geometry>
-    </collision>
-    <collision>
-      <origin xyz="-0.022 0.00 -0.27" rpy="0 -0.75 0" />
-      <geometry>
-        <box size="0.017 0.05 0.05" />
+      <origin xyz="-0.025 -0.003 -0.12" rpy="0 0.0 0" />
+      <geometry>
+        <box size="0.046 0.046 0.14" />
+      </geometry>
+    </collision>
+    <collision>
+      <origin xyz="-0.022 0.00 -0.275" rpy="0 -0.75 0" />
+      <geometry>
+        <box size="0.017 0.05 0.06" />
       </geometry>
     </collision>
@@ -228,7 +305,7 @@
   <link name="RL_calf">
     <inertial>
-      <origin xyz="12.515E-03 -0.024E-03 -117.649E-03" rpy="0 0 0" />
-      <mass value="0.361" />
-      <inertia ixx="3869.035E-06" ixy="-0.093E-06" ixz="298.636E-06" iyy="3945.295E-06" iyz="0.826E-06" izz="150.991E-06" />
+      <origin xyz="4.018E-03 17.411E-03 -232.283E-03" rpy="0 0 0" />
+      <mass value="1.751" />
+      <inertia ixx="14397.534E-06" ixy="124.726E-06" ixz="-550.242E-06" iyy="14603.730E-06" iyz="1307.539E-06" izz="1498.341E-06" />
     </inertial>
     <visual>
@@ -238,11 +315,17 @@
       </geometry>
       <material name="">
-        <color rgba="0.898039215686275 0.917647058823529 0.929411764705882 1" />
-      </material>
-    </visual>
-    <collision>
-      <origin xyz="0.018 -0.00 -0.08" rpy="0 -0.24 0" />
-      <geometry>
-        <box size="0.024 0.03 0.1" />
+        <color rgba="0.792156862745098 0.819607843137255 0.933333333333333 1" />
+      </material>
+    </visual>
+    <collision>
+      <origin xyz="0.0 0.0 -0.275" rpy="1.571 0 0" />
+      <geometry>
+        <cylinder radius="0.05" length="0.03" />
+      </geometry>
+    </collision>
+    <collision>
+      <origin xyz="0.02 -0.00 -0.08" rpy="0 -0.24 0" />
+      <geometry>
+        <box size="0.022 0.03 0.1" />
       </geometry>
     </collision>
@@ -254,13 +337,7 @@
     </collision>
     <collision>
-      <origin xyz="0.029 -0.00 -0.236" rpy="0 0.2 0" />
-      <geometry>
-        <box size="0.02 0.036 0.06" />
-      </geometry>
-    </collision>
-    <collision>
-      <origin xyz="0.008 -0.00 -0.23" rpy="0 0.68 0" />
-      <geometry>
-        <box size="0.01 0.036 0.06" />
+      <origin xyz="0.027 -0.00 -0.23" rpy="0 0.2 0" />
+      <geometry>
+        <box size="0.028 0.04 0.04" />
       </geometry>
     </collision>
@@ -273,4 +350,33 @@
     <limit lower="-2.77" upper="-0.54" effort="180.0" velocity="14.6667" />
   </joint>
+  <link name="RL_wheel">
+    <inertial>
+      <origin xyz="0E-03 51.080E-03 0E-03" rpy="0 0 0" />
+      <mass value="0.982" />
+      <inertia ixx="2435.762E-06" ixy="0E-06" ixz="0E-06" iyy="4581.589E-06" iyz="0E-06" izz="2435.762E-06" />
+    </inertial>
+    <visual>
+      <origin xyz="0 0 0" rpy="0 0 0" />
+      <geometry>
+        <mesh filename="package://a2w_description/meshes/left_hind_Link4.STL" />
+      </geometry>
+      <material name="">
+        <color rgba="0.792156862745098 0.819607843137255 0.933333333333333 1" />
+      </material>
+    </visual>
+    <collision>
+      <origin xyz="0 0.0494 0" rpy="1.5708 0 0" />
+      <geometry>
+        <cylinder radius="0.0948" length="0.050" />
+      </geometry>
+    </collision>
+  </link>
+  <joint name="RL_wheel_joint" type="${wheel_joint_type}">
+    <origin xyz="0 0 -0.275" rpy="0 0 0" />
+    <parent link="RL_calf" />
+    <child link="RL_wheel" />
+    <axis xyz="0 1 0" />
+    <limit effort="24.5" velocity="114.4" />
+  </joint>
   <link name="FR_hip">
     <inertial>
@@ -288,4 +394,16 @@
       </material>
     </visual>
+    <collision>
+      <origin xyz="0.0 -0.085 0" rpy="1.571 0 0" />
+      <geometry>
+        <cylinder radius="0.046" length="0.12" />
+      </geometry>
+    </collision>
+    <collision>
+      <origin xyz="0.0 -0.01 0" rpy="1.571 0 0" />
+      <geometry>
+        <cylinder radius="0.045" length="0.06" />
+      </geometry>
+    </collision>
   </link>
   <joint name="FR_hip_joint" type="${leg_joint_type}">
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